File: Powerboard/Hardware/redundantreg.kicad_sch (KiCad schematic)
At the start: 24 parts, among them Q10 MCH6351, Q9 MCH6351, U6 LM2679T-3.3-iclr, U7 LM2679T-3.3-iclr, U8 LTC4412xS6, U9 LTC4412xS6

Commit message: new board
Parts:
- removed C19, C20: 47uF, Capacitor_SMD:C_2220_5650Metric, symbol Device:C_Small
- removed C36, C37: 0.01uF, Capacitor_SMD:C_0603_1608Metric, symbol Device:C_Small
- removed C38, C39, C40, C41: 330uF, Capacitor_Tantalum_SMD:CP_EIA-7343-30_AVX-N, symbol Device:C_Polarized
- removed C42, C43: 0.47uF, Capacitor_SMD:C_0805_2012Metric, symbol Device:C_Small
- removed C44, C45: 22uF, Capacitor_SMD:C_0603_1608Metric, symbol Device:C_Small
- removed C48, C49: 0.1uF, Capacitor_SMD:C_0603_1608Metric, symbol Device:CP_Small
- removed D5, D6: DST1550S, Package_TO_SOT_SMD:TO-277B, symbol Device:D_Schottky_AAK
- removed L3, L4: 15uH, Inductor_SMD:L_12x12mm_H8mm, symbol iclr:P0846SNL-iclr
- removed Q10, Q9: MCH6351, Package_TO_SOT_SMD:SOT-363_SC-70-6, symbol iclr:MCH6351
- removed U6, U7: LM2679T-3.3-iclr, Package_TO_SOT_SMD:TO-263-7_TabPin4, symbol iclr:LM2679T-3.3-iclr
- removed U8, U9: LTC4412xS6, Package_TO_SOT_SMD:TSOT-23-6, symbol Power_Management:LTC4412xS6
- added C? (x4): 330uF, Capacitor_Tantalum_SMD:CP_EIA-7343-30_AVX-N, symbol Device:C_Polarized
- added C? (x2): 0.01uF, Capacitor_SMD:C_0603_1608Metric, symbol Device:C_Small
- added C? (x2): 220nF, symbol Device:C_Small
- added C? (x2): 22uF, Capacitor_SMD:C_0603_1608Metric, symbol Device:C_Small
- added C? (x2): 0.47uF, Capacitor_SMD:C_0805_2012Metric, symbol Device:C_Small
- added C? (x2): 1800uF, symbol Device:C_Small
- added C? (x2): 47uF, Capacitor_SMD:C_2220_5650Metric, symbol Device:C_Small
- added C? (x2): 0.1uF, Capacitor_SMD:C_0603_1608Metric, symbol Device:CP_Small
- added D? (x2): DST1550S, Package_TO_SOT_SMD:TO-277B, symbol Device:D_Schottky_AAK
- added L? (x2): 15uH, P0846SNL, symbol iclr:P0846SNL-iclr
- added Q? (x2): SSM6J511NU,LF, TRANS_SSM6J511NU,LF, symbol iclr:SSM6J511NU,LF
- added R? (x2): 6k8, symbol Device:R_Small
- added U? (x2): LTC4412xS6, Package_TO_SOT_SMD:TSOT-23-6, symbol Power_Management:LTC4412xS6
- added U? (x2): LM2679T-3.3-iclr, TO127P457X1016X2052-7P, symbol iclr:LM2679T-3.3-iclr
Connections:
- net GND: now also C?.2, C?.2, C?.2, C?.2, C?.2, C?.2, C?.2, C?.2, C?.2, C?.2, C?.2, C?.2, C?.2, C?.2, C?.2, C?.2, D?.1 (A), D?.1 (A), D?.2 (A), D?.2 (A), R?.2, R?.2, U?.2 (GND), U?.2 (GND), U?.3 (CTL), U?.3 (CTL), U?.4 (GND), U?.4 (GND)
- net STAT1: now also U?.4 (STAT)
- net STAT2: now also U?.4 (STAT)
- new net: C?.2, D?.3 (K), L?.1, U?.1 (SW) (x2)
- new net: C?.1, C?.1, C?.1, C?.1, L?.2, Q?.1, Q?.2, Q?.5, Q?.6, Q?.7, U?.1 (VIN), U?.6 (FB) (x2)
- new net: C?.1, U?.3 (BOOST) (x2)
- new net: C?.1, U?.7 (SOFTSTART) (x2)
- new net: R?.1, U?.5 (CURRENT_ADJ) (x2)
- new net: Q?.3, U?.5 (GATE) (x2)
- new net +12V: C?.1, C?.1, C?.1, C?.1, U?.2 (VIN), U?.2 (VIN)
- new net +3V3: C?.1, C?.1, Q?.4, Q?.4, Q?.8, Q?.8, U?.6 (SENSE), U?.6 (SENSE)
- no-connect marks 2 -> 0
Other:
- note added: "0.127uF using calculation. Data sheet says standard value of 0.22uF is also acceptable."
