File: Powerboard/Hardware/usb__uart.kicad_sch (KiCad schematic)
At the start: 23 parts, among them IC2 CP2102, J8 USB_C_Receptacle_USB2.0, U11 LTC4411, U4 SC4216H

Commit message: new board
Parts:
- removed C50: 1.0uF, Capacitor_SMD:C_0603_1608Metric, symbol Device:C_Small
- removed C51, C53: 0.1uF, Capacitor_SMD:C_0603_1608Metric, symbol Device:C_Small
- removed C52, C58: 4.7uF, Capacitor_SMD:C_0603_1608Metric, symbol Device:C_Small
- removed C54, C57: 10uF, Capacitor_SMD:C_0603_1608Metric, symbol Device:C_Small
- removed D7: LED, LED_SMD:LED_0603_1608Metric, symbol Device:LED
- removed D8: SP0503BAHT, Package_TO_SOT_SMD:SOT-143, symbol Power_Protection:SP0503BAHT
- removed IC2: CP2102, iclr:QFN28G_0.5-5X5MM, symbol iclr:CP2102
- removed J8: USB_C_Receptacle_USB2.0, Connector_USB:USB_C_Receptacle_GCT_USB4085, symbol Connector:USB_C_Receptacle_USB2.0
- removed R35, R36: 5.1k, Resistor_SMD:R_0603_1608Metric, symbol Device:R_Small
- removed R37: 470, Resistor_SMD:R_0603_1608Metric, symbol Device:R_Small
- removed R38: 24k, Resistor_SMD:R_0603_1608Metric, symbol Device:R_Small
- removed R39: 47k, Resistor_SMD:R_0603_1608Metric, symbol Device:R_Small
- removed R40: 4.7k, Resistor_SMD:R_0603_1608Metric, symbol Device:R_Small
- removed R42: 56k, Resistor_SMD:R_0603_1608Metric, symbol Device:R_Small
- removed R43: 10k, Resistor_SMD:R_0603_1608Metric, symbol Device:R_Small
- removed TP23, TP24: TestPoint, TestPoint:TestPoint_Pad_D1.0mm, symbol Connector:TestPoint
- removed U11: LTC4411, Package_TO_SOT_SMD:SOT-23-5, symbol iclr:LTC4411
- removed U4: SC4216H, iclr:SOIC127P599X175-9N, symbol iclr:RT9025-25GSP
Connections:
- no-connect marks 22 -> 0
