File: Powerboard/Hardware/usb-uart.kicad_sch (KiCad schematic)
At the start: 16 parts, among them J3 USB_C_Receptacle_USB2.0, U3 SC4216H, U4 LTC4411

Commit message: latest
Parts:
- removed C15, C16: 10uF, Capacitor_SMD:C_0603_1608Metric, symbol Device:C_Small
- removed D1: SP0503BAHT, Package_TO_SOT_SMD:SOT-143, symbol Power_Protection:SP0503BAHT
- removed J3: USB_C_Receptacle_USB2.0, Connector_USB:USB_C_Receptacle_GCT_USB4085, symbol Connector:USB_C_Receptacle_USB2.0
- removed R10, R11: 5.1k, Resistor_SMD:R_0402_1005Metric, symbol Device:R_Small
- removed R14: 10k, Resistor_SMD:R_0402_1005Metric, symbol Device:R_Small
- removed TP1, TP2, TP3: TestPoint, TestPoint:TestPoint_Pad_D1.0mm, symbol Connector:TestPoint
- removed U3: SC4216H, iclr:SOIC127P599X175-9N, symbol iclr:RT9025-25GSP
- removed U4: LTC4411, Package_TO_SOT_SMD:SOT-23-5, symbol iclr:LTC4411
- added C49: 1uF, Capacitor_SMD:C_0402_1005Metric, symbol Device:C_Small
- added C50: 22uF, Capacitor_SMD:C_0603_1608Metric, symbol Device:C_Small
- added C51, C53: 10uF, Capacitor_SMD:C_0402_1005Metric, symbol Device:C_Small
- added C52: 4.7uF, Capacitor_SMD:C_0402_1005Metric, symbol Device:C_Small
- added C54: 0.1uF, Capacitor_SMD:C_0402_1005Metric, symbol Device:C_Small
- added L5: 1uH, Inductor_SMD:L_0805_2012Metric, symbol Device:L
- added R1: 14k, Resistor_SMD:R_0402_1005Metric, symbol Device:R_Small
- added R2: 56k, Resistor_SMD:R_0402_1005Metric, symbol Device:R_Small
- added TP4: TestPoint, TestPoint:TestPoint_Pad_D1.5mm, symbol Connector:TestPoint
- added U10: SC4215, iclr:SOIC127P599X175-9N, symbol iclr:RT9025-25GSP
- added U4: MAX77827AEFD+T, iclr:CONV_MAX77827AEFD+T, symbol iclr:MAX77827AEFD+T
- C17: value 4.7uF -> 10uF
- R13: value 56k -> 10k
Connections:
- net GND: now also R13.2, C50.2, C51.2, C52.2, C53.1, C54.1, U10.8 (GND), U10.9 (GND), U4.9 (PGND)
- net FBIn: now reaches R13.1
- net FBIn: now also R2.2, U10.7 (ADJ)
- net 3.3V renamed RBUS_uC_V
- net RBUS_uC_V: now also TP4.1, U4.3 (EN), U4.6 (IN)
- new net +3V3: C53.2, C54.2, R2.1, U10.6 (VOUT)
- new net BBOUT: C50.1, C51.1, C52.1, U10.2 (EN), U10.3 (VIN), U4.11 (OUT), U4.13 (OUTS)
- new net BIAS: C49.1, U4.5 (BIAS)
- new net GNDA: C49.2, R1.2, U4.4 (AGND)
- new net LX1: L5.1, U4.8 (LX1)
- new net LX2: L5.2, U4.10 (LX2)
- new net SEL: R1.1, U4.1 (SEL)
- no-connect marks 5 -> 4
Other:
- moved on the sheet: R12, USBLED1

Commit message: waiting for review
Parts:
- removed TP4: TestPoint, TestPoint:TestPoint_Pad_D1.5mm, symbol Connector:TestPoint
- USBLED1: footprint LED_SMD:LED_0603_1608Metric -> LED_SMD:LED_0402_1005Metric
Changed lines of the file:
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@@
   (junction (at 242.062 69.85) (diameter 0) (color 0 0 0 0)
-  )
-  (junction (at 109.982 69.85) (diameter 0) (color 0 0 0 0)
   )
   (junction (at 170.942 69.85) (diameter 0) (color 0 0 0 0)
@@
     (stroke (width 0) (type default) (color 0 0 0 0))
   )
-  (wire (pts (xy 109.982 69.85) (xy 115.062 69.85))
+  (wire (pts (xy 96.52 69.85) (xy 115.062 69.85))
     (stroke (width 0) (type default) (color 0 0 0 0))
   )
@@
   )
   (wire (pts (xy 226.822 69.85) (xy 239.522 69.85))
-    (stroke (width 0) (type default) (color 0 0 0 0))
-  )
-  (wire (pts (xy 96.52 69.85) (xy 109.982 69.85))
     (stroke (width 0) (type default) (color 0 0 0 0))
   )
@@
     (property "Reference" "USBLED1" (id 0) (at 145.034 99.949 0))
     (property "Value" "USB_LED" (id 1) (at 145.034 102.2604 0))
-    (property "Footprint" "LED_SMD:LED_0603_1608Metric" (id 2) (at 145.034 105.156 90)
+    (property "Footprint" "LED_SMD:LED_0402_1005Metric" (id 2) (at 145.034 105.156 90)
       (effects (font (size 1.27 1.27)) hide)
     )
@@
     (pin "9")
   )
-  (symbol (lib_id "Connector:TestPoint") (at 109.982 69.85 0) (unit 1)
-    (in_bom yes) (on_board yes)
-    (property "Reference" "TP4" (id 0) (at 108.712 63.5 0)
-      (effects (font (size 1.27 1.27)) (justify left))
-    )
-    (property "Value" "TestPoint" (id 1) (at 108.712 60.9631 0)
-      (effects (font (size 1.27 1.27)) (justify left))
-    )
-    (property "Footprint" "TestPoint:TestPoint_Pad_D1.5mm" (id 2) (at 115.062 69.85 0)
-      (effects (font (size 1.27 1.27)) hide)
-    )
-    (property "Datasheet" "~" (id 3) (at 115.062 69.85 0)
-      (effects (font (size 1.27 1.27)) hide)
-    )
-    (pin "1")
-  )
   (symbol (lib_id "power:GNDA") (at 118.872 90.17 0) (unit 1)

Commit message: kiran/andrei review
Parts:
- added TP3: TestPoint, TestPoint:TestPoint_Pad_D1.0mm, symbol Connector:TestPoint
Connections:
- net RBUS_uC_V: now also TP3.1
Changed lines of the file:
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@@
   (junction (at 187.452 69.85) (diameter 0) (color 0 0 0 0)
+  )
+  (junction (at 107.696 69.85) (diameter 0) (color 0 0 0 0)
   )
   (junction (at 242.062 69.85) (diameter 0) (color 0 0 0 0)
@@
     (stroke (width 0) (type default))
   )
-  (wire (pts (xy 96.52 69.85) (xy 115.062 69.85))
+  (wire (pts (xy 96.52 69.85) (xy 107.696 69.85))
     (stroke (width 0) (type default))
   )
@@
   )
   (wire (pts (xy 112.522 82.55) (xy 122.682 82.55))
+    (stroke (width 0) (type default))
+  )
+  (wire (pts (xy 107.696 69.85) (xy 115.062 69.85))
     (stroke (width 0) (type default))
   )
@@
         )
       )
+    )
+  )
+  (symbol (lib_id "Connector:TestPoint") (at 107.696 69.85 0) (unit 1)
+    (in_bom yes) (on_board yes) (dnp no) (fields_autoplaced)
+    (property "Reference" "TP3" (at 109.093 65.9043 0)
+      (effects (font (size 1.27 1.27)) (justify left))
+    )
+    (property "Value" "TestPoint" (at 109.093 67.8253 0)
+      (effects (font (size 1.27 1.27)) (justify left))
+    )
+    (property "Footprint" "TestPoint:TestPoint_Pad_D1.0mm" (at 112.776 69.85 0)
+      (effects (font (size 1.27 1.27)) hide)
+    )
+    (property "Datasheet" "~" (at 112.776 69.85 0)
+      (effects (font (size 1.27 1.27)) hide)
+    )
+    (pin "1")
+    (instances
+      (project "Switcher"
+        (path "/e63e39d7-6ac0-4ffd-8aa3-1841a4541b55/12e3318b-d723-448e-80f4-0a2add1fb722"
+          (reference "TP3") (unit 1)
+        )
+      )
