File: Powerboard/Hardware/Switcher.kicad_sch (KiCad schematic)
At the start: 40 parts, among them J1 Conn_01x03_MountingPin, J2 Conn_01x02_Male, U1 SN74LVC1G373DCKR, U2 ESP32-S3, Y1 40MHz±10ppm

Commit message: latest
Parts:
- removed J2: Conn_01x02_Male, Connector_Molex:Molex_Nano-Fit_105313-xx02_1x02_P2.50mm_Horizontal, symbol Connector:Conn_01x02_Male
- removed R1, R2: R_Small, Resistor_SMD:R_0402_1005Metric, symbol Device:R_Small
- removed RXLED1: RX_LED, LED_SMD:LED_0603_1608Metric, symbol Device:LED_Small
- removed U1: SN74LVC1G373DCKR, iclr:SOT65P210X110-6N, symbol iclr:SN74LVC1G373DCKR
- added J2: XT60PW-F, iclr:AMASS_XT60PW-F, symbol iclr:XT60PW-F
- added J7: XT60PW-M, iclr:AMASS_XT60PW-M, symbol iclr:XT60PW-M
- C12: value C -> 4.2pF
- R4: value 470 -> 499
- R8: value 50 -> 47.5
Connections:
- net +12V: now also J2.1
- net +3V3: no longer R4.1
- net GND: now also J7.2 (-)
- net PDU_EN: now also J1.1 (Pin_1), U2.30 (SPIHD/GPIO27)
- net TXD: now also R4.1
- net at R4.2: now also U2.49 (U0TXD/PROG/GPIO43)
- net USBPOWER: now reaches U2.36 (SPICLK_N/GPIO48)
- net LIPOPOWER: now reaches U2.37 (SPICLK_P/GPIO47)
- new net: J2.2, J7.1 (+)
- new net: J2.S1 (SHIELD), J2.S2 (SHIELD)
- no-connect marks 36 -> 33
Other:
- sheet 3V3Bucks renamed Bucks
- added sheet 3V3Filter (usb-uart.kicad_sch)
- sheet Bucks ports: added LIPOPOWER, USBPOWER; removed STAT1, STAT2
- sheet USB: file usb-uart.kicad_sch -> untitled.kicad_sch
- sheet USB ports: added none; removed 3.3V

Commit message: added power rail logging
Parts:
- added R14: 47k, Resistor_SMD:R_0402_1005Metric, symbol Device:R_Small
- added R22: 10k, Resistor_SMD:R_0402_1005Metric, symbol Device:R_Small
Connections:
- net +12V: now also R14.1
- net GND: now also R22.2
- net DeploymentVoltage: now reaches U2.27 (GPIO21)
- net DeploymentVoltage: now also R14.2, R22.1
- no-connect marks 33 -> 32
Changed lines of the file:
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@@
   (junction (at 165.862 148.082) (diameter 0) (color 0 0 0 0)
+  )
+  (junction (at 61.468 148.844) (diameter 0) (color 0 0 0 0)
   )
   (junction (at 47.498 183.896) (diameter 0) (color 0 0 0 0)
@@
   (no_connect (at 242.062 70.612))
   (no_connect (at 242.062 73.152))
-  (no_connect (at 242.062 75.692))
   (no_connect (at 242.062 78.232))
   (no_connect (at 242.062 83.312))
@@
     (stroke (width 0) (type default) (color 0 0 0 0))
   )
+  (wire (pts (xy 61.468 147.574) (xy 61.468 148.844))
+    (stroke (width 0) (type default) (color 0 0 0 0))
+  )
   (wire (pts (xy 249.682 139.192) (xy 262.382 139.192))
     (stroke (width 0) (type default) (color 0 0 0 0))
@@
     (stroke (width 0) (type default) (color 0 0 0 0))
   )
+  (wire (pts (xy 61.468 148.844) (xy 61.468 149.86))
+    (stroke (width 0) (type default) (color 0 0 0 0))
+  )
   (wire (pts (xy 242.062 62.992) (xy 250.952 62.992))
     (stroke (width 0) (type default) (color 0 0 0 0))
@@
   )
   (wire (pts (xy 140.462 165.862) (xy 143.002 165.862))
+    (stroke (width 0) (type default) (color 0 0 0 0))
+  )
+  (wire (pts (xy 61.468 148.844) (xy 65.786 148.844))
     (stroke (width 0) (type default) (color 0 0 0 0))
   )
@@
     (effects (font (size 1.27 1.27)) (justify right bottom))
   )
+  (label "DeploymentVoltage" (at 65.786 148.844 0)
+    (effects (font (size 1.27 1.27)) (justify left bottom))
+  )
   (label "BOOT" (at 159.512 192.532 180)
     (effects (font (size 1.27 1.27)) (justify right bottom))
+  )
+  (label "DeploymentVoltage" (at 242.062 75.692 0)
+    (effects (font (size 1.27 1.27)) (justify left bottom))
   )
   (label "CHIP_PU" (at 143.002 165.862 180)
@@
     )
     (property "Datasheet" "" (id 3) (at 126.492 136.652 0)
+      (effects (font (size 1.27 1.27)) hide)
+    )
+    (pin "1")
+  )
+  (symbol (lib_id "power:GND") (at 61.468 154.94 0) (unit 1)
+    (in_bom yes) (on_board yes)
+    (property "Reference" "#PWR0141" (id 0) (at 61.468 161.29 0)
+      (effects (font (size 1.27 1.27)) hide)
+    )
+    (property "Value" "GND" (id 1) (at 61.595 159.3342 0))
+    (property "Footprint" "" (id 2) (at 61.468 154.94 0)
+      (effects (font (size 1.27 1.27)) hide)
+    )
+    (property "Datasheet" "" (id 3) (at 61.468 154.94 0)
       (effects (font (size 1.27 1.27)) hide)
     )
@@
     (pin "2")
   )
+  (symbol (lib_id "Device:R_Small") (at 61.468 152.4 0) (unit 1)
+    (in_bom yes) (on_board yes) (fields_autoplaced)
+    (property "Reference" "R22" (id 0) (at 62.9666 151.5653 0)
+      (effects (font (size 1.27 1.27)) (justify left))
+    )
+    (property "Value" "10k" (id 1) (at 62.9666 154.1022 0)
+      (effects (font (size 1.27 1.27)) (justify left))
+    )
+    (property "Footprint" "Resistor_SMD:R_0402_1005Metric" (id 2) (at 61.468 152.4 0)
+      (effects (font (size 1.27 1.27)) hide)
+    )
+    (property "Datasheet" "~" (id 3) (at 61.468 152.4 0)
+      (effects (font (size 1.27 1.27)) hide)
+    )
+    (pin "1")
+    (pin "2")
+  )
   (symbol (lib_id "Device:C_Small") (at 160.782 170.942 270) (unit 1)
     (in_bom yes) (on_board yes)
@@
     )
     (pin "1")
+  )
+  (symbol (lib_id "Device:R_Small") (at 61.468 145.034 0) (unit 1)
+    (in_bom yes) (on_board yes) (fields_autoplaced)
+    (property "Reference" "R14" (id 0) (at 62.9666 144.1993 0)
+      (effects (font (size 1.27 1.27)) (justify left))
+    )
+    (property "Value" "47k" (id 1) (at 62.9666 146.7362 0)
+      (effects (font (size 1.27 1.27)) (justify left))
+    )
+    (property "Footprint" "Resistor_SMD:R_0402_1005Metric" (id 2) (at 61.468 145.034 0)
+      (effects (font (size 1.27 1.27)) hide)
+    )
+    (property "Datasheet" "~" (id 3) (at 61.468 145.034 0)
+      (effects (font (size 1.27 1.27)) hide)
+    )
+    (pin "1")
+    (pin "2")
   )
   (symbol (lib_id "Device:R_Small") (at 151.892 188.722 0) (unit 1)
@@
     (pin "1")
   )
+  (symbol (lib_id "power:+12V") (at 61.468 142.494 0) (unit 1)
+    (in_bom yes) (on_board yes) (fields_autoplaced)
+    (property "Reference" "#PWR0135" (id 0) (at 61.468 146.304 0)
+      (effects (font (size 1.27 1.27)) hide)
+    )
+    (property "Value" "+12V" (id 1) (at 61.468 138.9182 0))
+    (property "Footprint" "" (id 2) (at 61.468 142.494 0)
+      (effects (font (size 1.27 1.27)) hide)
+    )
+    (property "Datasheet" "" (id 3) (at 61.468 142.494 0)
+      (effects (font (size 1.27 1.27)) hide)
+    )
+    (pin "1")
+  )
   (symbol (lib_id "Device:C_Small") (at 135.382 139.192 0) (unit 1)
     (in_bom yes) (on_board yes)
@@
       (reference "#PWR0134") (unit 1) (value "VBUS") (footprint "")
     )
+    (path "/90dd16e7-d068-412a-b518-16a1e9fa0d08"
+      (reference "#PWR0135") (unit 1) (value "+12V") (footprint "")
+    )
     (path "/12646a0c-a158-4f1c-9172-cd278d717c5e/5d9baebe-2425-45d7-8700-e8094c810011"
       (reference "#PWR0136") (unit 1) (value "GND") (footprint "")
@@
       (reference "#PWR0140") (unit 1) (value "GND") (footprint "")
     )
+    (path "/0c43492a-1d06-42e1-aab3-dafca109a963"
+      (reference "#PWR0141") (unit 1) (value "GND") (footprint "")
+    )
     (path "/133f56f4-a29c-4cbf-87b7-9d99a292e3c0/932f22b3-e743-4b9a-8d98-03e3af0a31b4"
       (reference "#PWR0142") (unit 1) (value "GND") (footprint "")
@@
       (reference "R13") (unit 1) (value "10k") (footprint "Resistor_SMD:R_0402_1005Metric")
     )
+    (path "/53c0fa19-4857-45ef-a0b0-d2d75f95cdd8"
+      (reference "R14") (unit 1) (value "47k") (footprint "Resistor_SMD:R_0402_1005Metric")
+    )
     (path "/12646a0c-a158-4f1c-9172-cd278d717c5e/2b8f9035-c4ba-4acb-8c8e-2b186e0ff025"
       (reference "R15") (unit 1) (value "10k") (footprint "Resistor_SMD:R_0402_1005Metric")
@@
       (reference "R21") (unit 1) (value "10k") (footprint "Resistor_SMD:R_0402_1005Metric")
     )
+    (path "/3ae3fbd7-43c3-40f9-ba93-33b016cd17e5"
+      (reference "R22") (unit 1) (value "10k") (footprint "Resistor_SMD:R_0402_1005Metric")
+    )
     (path "/e469982c-3823-4665-9e6d-e90b00c2da09/518041de-f29f-4e9d-8826-cb8f5467094e"

Commit message: waiting for review
Connections:
- net +12V: now also J2.2; no longer J2.1
- net GND: now also J7.1 (+); no longer J7.2 (-)
- new net: J2.1, J7.2 (-)
Changed lines of the file:
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@@
-    (stroke (width 0) (type default) (color 0 0 0 0))
-  )
-  (wire (pts (xy 235.966 29.21) (xy 239.014 29.21))
     (stroke (width 0) (type default) (color 0 0 0 0))
   )
@@
     (stroke (width 0) (type default) (color 0 0 0 0))
   )
-  (wire (pts (xy 223.52 29.21) (xy 223.52 31.75))
-    (stroke (width 0) (type default) (color 0 0 0 0))
-  )
   (wire (pts (xy 165.862 62.992) (xy 169.672 62.992))
     (stroke (width 0) (type default) (color 0 0 0 0))
@@
     (stroke (width 0) (type default) (color 0 0 0 0))
   )
-  (wire (pts (xy 223.52 29.21) (xy 233.426 29.21))
-    (stroke (width 0) (type default) (color 0 0 0 0))
-  )
-  (wire (pts (xy 226.06 25.4) (xy 226.06 31.75))
-    (stroke (width 0) (type default) (color 0 0 0 0))
-  )
   (wire (pts (xy 159.512 192.532) (xy 151.892 192.532))
     (stroke (width 0) (type default) (color 0 0 0 0))
@@
     (stroke (width 0) (type default) (color 0 0 0 0))
   )
-  (wire (pts (xy 239.014 29.21) (xy 239.014 30.734))
-    (stroke (width 0) (type default) (color 0 0 0 0))
-  )
   (wire (pts (xy 174.752 165.862) (xy 169.672 165.862))
     (stroke (width 0) (type default) (color 0 0 0 0))
@@
     (stroke (width 0) (type default) (color 0 0 0 0))
   )
+  (wire (pts (xy 235.966 31.75) (xy 235.966 29.21))
+    (stroke (width 0) (type default) (color 0 0 0 0))
+  )
   (wire (pts (xy 61.468 148.844) (xy 61.468 149.86))
     (stroke (width 0) (type default) (color 0 0 0 0))
@@
   )
   (wire (pts (xy 140.462 165.862) (xy 143.002 165.862))
+    (stroke (width 0) (type default) (color 0 0 0 0))
+  )
+  (wire (pts (xy 226.06 31.75) (xy 235.966 31.75))
     (stroke (width 0) (type default) (color 0 0 0 0))
   )
@@
     (pin "2")
   )
-  (symbol (lib_id "power:+12V") (at 226.06 25.4 0) (unit 1)
-    (in_bom yes) (on_board yes)
-    (property "Reference" "#PWR0184" (id 0) (at 226.06 29.21 0)
-      (effects (font (size 1.27 1.27)) hide)
-    )
-    (property "Value" "+12V" (id 1) (at 226.06 20.32 0))
-    (property "Footprint" "" (id 2) (at 226.06 25.4 0)
-      (effects (font (size 1.27 1.27)) hide)
-    )
-    (property "Datasheet" "" (id 3) (at 226.06 25.4 0)
+  (symbol (lib_id "power:+12V") (at 223.52 31.75 0) (unit 1)
+    (in_bom yes) (on_board yes)
+    (property "Reference" "#PWR0184" (id 0) (at 223.52 35.56 0)
+      (effects (font (size 1.27 1.27)) hide)
+    )
+    (property "Value" "+12V" (id 1) (at 223.52 26.67 0))
+    (property "Footprint" "" (id 2) (at 223.52 31.75 0)
+      (effects (font (size 1.27 1.27)) hide)
+    )
+    (property "Datasheet" "" (id 3) (at 223.52 31.75 0)
       (effects (font (size 1.27 1.27)) hide)
     )
@@
     (pin "1")
   )
-  (symbol (lib_id "power:GND") (at 239.014 30.734 0) (unit 1)
+  (symbol (lib_id "power:GND") (at 233.426 29.21 0) (unit 1)
     (in_bom yes) (on_board yes) (fields_autoplaced)
-    (property "Reference" "#PWR0185" (id 0) (at 239.014 37.084 0)
-      (effects (font (size 1.27 1.27)) hide)
-    )
-    (property "Value" "GND" (id 1) (at 239.014 35.1774 0))
-    (property "Footprint" "" (id 2) (at 239.014 30.734 0)
-      (effects (font (size 1.27 1.27)) hide)
-    )
-    (property "Datasheet" "" (id 3) (at 239.014 30.734 0)
+    (property "Reference" "#PWR0185" (id 0) (at 233.426 35.56 0)
+      (effects (font (size 1.27 1.27)) hide)
+    )
+    (property "Value" "GND" (id 1) (at 233.426 33.6534 0))
+    (property "Footprint" "" (id 2) (at 233.426 29.21 0)
+      (effects (font (size 1.27 1.27)) hide)
+    )
+    (property "Datasheet" "" (id 3) (at 233.426 29.21 0)
       (effects (font (size 1.27 1.27)) hide)
     )
@@
     )
     (path "/7369ceff-38ea-4740-9245-fda19d5ff608/871d6184-92c3-46ec-bb43-46ca046825fc"
-      (reference "J3") (unit 1) (value "USB_C_Receptacle_USB2.0") (footprint "Connector_USB:USB_C_Receptacle_GCT_USB4085")
+      (reference "J3") (unit 1) (value "USB_C_Receptacle_USB2.0") (footprint "Connector_USB:USB_C_Receptacle_Palconn_UTC16-G")
     )
     (path "/133f56f4-a29c-4cbf-87b7-9d99a292e3c0/031213dd-5689-4d36-a614-00163f71bac8"
@@
       (reference "J7") (unit 1) (value "XT60PW-M") (footprint "iclr:AMASS_XT60PW-M")
     )
-    (path "/12646a0c-a158-4f1c-9172-cd278d717c5e/d6a951f9-4e8e-48ab-9754-144240f34c5b"
-      (reference "JP1") (unit 1) (value "TermJP") (footprint "Jumper:SolderJumper-3_P1.3mm_Open_RoundedPad1.0x1.5mm")
-    )
     (path "/133f56f4-a29c-4cbf-87b7-9d99a292e3c0/0c7d0a88-501b-4135-9470-5cf02591d1ed"
       (reference "JP2") (unit 1) (value "SolderJumper_2_Bridged") (footprint "Jumper:SolderJumper-2_P1.3mm_Bridged_RoundedPad1.0x1.5mm")
@@
       (reference "R22") (unit 1) (value "10k") (footprint "Resistor_SMD:R_0402_1005Metric")
     )
+    (path "/12646a0c-a158-4f1c-9172-cd278d717c5e/a3befb04-ad83-4d71-93e6-31a252aa254c"
+      (reference "R23") (unit 1) (value "0") (footprint "Resistor_SMD:R_0402_1005Metric")
+    )
     (path "/e469982c-3823-4665-9e6d-e90b00c2da09/518041de-f29f-4e9d-8826-cb8f5467094e"
       (reference "R25") (unit 1) (value "100k") (footprint "Resistor_SMD:R_0402_1005Metric")
@@
       (reference "TP2") (unit 1) (value "TestPoint") (footprint "TestPoint:TestPoint_Pad_D1.0mm")
     )
-    (path "/7369ceff-38ea-4740-9245-fda19d5ff608/3d13a3de-a04e-47e4-8b79-1d1816e873cf"
-      (reference "TP3") (unit 1) (value "TestPoint") (footprint "TestPoint:TestPoint_Pad_D1.0mm")
-    )
-    (path "/12e3318b-d723-448e-80f4-0a2add1fb722/4bbf6873-85fa-4780-87de-d6d500e2d77b"
-      (reference "TP4") (unit 1) (value "TestPoint") (footprint "TestPoint:TestPoint_Pad_D1.5mm")
-    )
     (path "/f73ce9e8-73f6-4662-b9bd-23c6fb5e51dd"
       (reference "TXLED1") (unit 1) (value "TX_LED") (footprint "Resistor_SMD:R_0402_1005Metric")
@@
     )
     (path "/12e3318b-d723-448e-80f4-0a2add1fb722/3493ab04-6e23-41d0-b5c5-6b75aa90f2b5"
-      (reference "USBLED1") (unit 1) (value "USB_LED") (footprint "LED_SMD:LED_0603_1608Metric")
+      (reference "USBLED1") (unit 1) (value "USB_LED") (footprint "LED_SMD:LED_0402_1005Metric")
     )
     (path "/67b54d4e-5a74-4132-b615-efac7c8baddf"

Commit message: i2c breakout, general clean up
Parts:
- added J8: Conn_01x04_Male, Connector_PinHeader_2.54mm:PinHeader_1x04_P2.54mm_Vertical, symbol Connector:Conn_01x04_Male
- J1: footprint Connector_Molex:Molex_Nano-Fit_105313-xx02_1x02_P2.50mm_Horizontal -> iclr:Molex_Nano-Fit_105313-xx02_1x02_P2.50mm_Horizontal
- U2: footprint Package_DFN_QFN:QFN-56-1EP_7x7mm_P0.4mm_EP5.6x5.6mm -> iclr:QFN40P700X700X90-57N
Connections:
- net +3V3: now also J8.1 (Pin_1)
- net GND: now also J8.2 (Pin_2)
- net 3.3STAT1 renamed SDA
- net SDA: now also J8.4 (Pin_4)
- net 3.3STAT2 renamed SCL
- net SCL: now also J8.3 (Pin_3)

Commit message: vias fixed, ready for review
Connections:
- net SCL: now also U2.44 (MTCK/JTAG/GPIO39); no longer U2.43 (GPIO38)
- net SDA: now also U2.43 (GPIO38); no longer U2.44 (MTCK/JTAG/GPIO39)
- net LATCH_STAT renamed 3V3LOG
Other:
- sheet Switches+RBUS ports: added 3V3LOG; removed none
Changed lines of the file:
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@@
     (effects (font (size 1.27 1.27)) (justify left bottom))
-  )
-  (label "LATCH_STAT" (at 176.022 126.492 180) (fields_autoplaced)
-    (effects (font (size 1.27 1.27)) (justify right bottom))
   )
   (label "LIPOPOWER" (at 242.062 118.872 0) (fields_autoplaced)
@@
     (effects (font (size 1.27 1.27)) (justify left bottom))
   )
+  (label "3V3LOG" (at 35.052 84.328 180) (fields_autoplaced)
+    (effects (font (size 1.27 1.27)) (justify right bottom))
+  )
   (label "SCL" (at 96.012 167.132 0) (fields_autoplaced)
     (effects (font (size 1.27 1.27)) (justify left bottom))
@@
     (effects (font (size 1.27 1.27)) (justify right bottom))
   )
-  (label "SCL" (at 242.062 108.712 0) (fields_autoplaced)
-    (effects (font (size 1.27 1.27)) (justify left bottom))
+  (label "SCL" (at 176.022 118.872 180) (fields_autoplaced)
+    (effects (font (size 1.27 1.27)) (justify right bottom))
   )
   (label "12V_SWITCH" (at 242.062 106.172 0) (fields_autoplaced)
@@
     (effects (font (size 1.27 1.27)) (justify left bottom))
   )
-  (label "SDA" (at 176.022 118.872 180) (fields_autoplaced)
+  (label "SDA" (at 242.062 108.712 0) (fields_autoplaced)
+    (effects (font (size 1.27 1.27)) (justify left bottom))
+  )
+  (label "3V3LOG" (at 176.022 126.492 180) (fields_autoplaced)
     (effects (font (size 1.27 1.27)) (justify right bottom))
   )
@@
       (effects (font (size 1.27 1.27)) (justify left))
     )
+    (pin "3V3LOG" input (at 35.052 84.328 180)
+      (effects (font (size 1.27 1.27)) (justify left))
+    )

Commit message: kiran/andrei review
Connections:
- net +3V3: now also J8.2 (Pin_2); no longer J8.1 (Pin_1)
- net GND: now also J8.1 (Pin_1); no longer J8.2 (Pin_2)
Changed lines of the file:
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@@
+    (stroke (width 0) (type default))
+  )
+  (wire (pts (xy 96.012 164.592) (xy 98.298 164.592))
     (stroke (width 0) (type default))
   )
@@
     (stroke (width 0) (type default))
   )
+  (wire (pts (xy 96.012 161.29) (xy 96.012 162.052))
+    (stroke (width 0) (type default))
+  )
   (wire (pts (xy 126.492 141.732) (xy 135.382 141.732))
     (stroke (width 0) (type default))
@@
     (stroke (width 0) (type default))
   )
-  (wire (pts (xy 96.012 164.592) (xy 103.124 164.592))
-    (stroke (width 0) (type default))
-  )
   (wire (pts (xy 123.952 31.242) (xy 129.032 31.242))
     (stroke (width 0) (type default))
@@
     (stroke (width 0) (type default))
   )
-  (wire (pts (xy 103.124 164.592) (xy 103.124 165.354))
+  (wire (pts (xy 103.124 161.29) (xy 103.124 165.354))
     (stroke (width 0) (type default))
   )
@@
     (stroke (width 0) (type default))
   )
+  (wire (pts (xy 103.124 161.29) (xy 96.012 161.29))
+    (stroke (width 0) (type default))
+  )
   (wire (pts (xy 151.892 170.942) (xy 151.892 172.212))
     (stroke (width 0) (type default))
@@
   )
   (polyline (pts (xy 230.632 112.522) (xy 230.632 115.062))
+    (stroke (width 0) (type default))
+  )
+  (wire (pts (xy 98.298 164.592) (xy 98.298 164.338))
     (stroke (width 0) (type default))
   )
@@
     )
   )
-  (symbol (lib_id "power:+3.3V") (at 96.012 162.052 0) (unit 1)
-    (in_bom yes) (on_board yes) (dnp no)
-    (property "Reference" "#PWR0155" (at 96.012 165.862 0)
-      (effects (font (size 1.27 1.27)) hide)
-    )
-    (property "Value" "+3.3V" (at 96.393 157.6578 0)
-      (effects (font (size 1.27 1.27)))
-    )
-    (property "Footprint" "" (at 96.012 162.052 0)
-      (effects (font (size 1.27 1.27)) hide)
-    )
-    (property "Datasheet" "" (at 96.012 162.052 0)
-      (effects (font (size 1.27 1.27)) hide)
-    )
+  (symbol (lib_id "power:+3.3V") (at 98.298 164.338 0) (unit 1)
+    (in_bom yes) (on_board yes) (dnp no)
+    (property "Reference" "#PWR0155" (at 98.298 168.148 0)
+      (effects (font (size 1.27 1.27)) hide)
+    )
+    (property "Value" "+3.3V" (at 98.679 159.9438 0)
+      (effects (font (size 1.27 1.27)))
+    )
+    (property "Footprint" "" (at 98.298 164.338 0)
+      (effects (font (size 1.27 1.27)) hide)
+    )
+    (property "Datasheet" "" (at 98.298 164.338 0)
+      (effects (font (size 1.27 1.27)) hide)
+    )
