File: Powerboard/Hardware/Switcher.kicad_sch (KiCad schematic)
At the start: 42 parts, among them J1 Conn_01x03_MountingPin, J2 XT60PW-F, J7 XT60PW-M, J8 Conn_01x04_Male, U2 ESP32-S3, Y1 40MHz±10ppm

Commit message: reviewed
Parts:
- C13, C14: footprint Capacitor_SMD:C_0603_1608Metric -> Capacitor_SMD:C_0402_1005Metric
Connections:
- net PDU_EN: now also U2.38 (GPIO33); no longer U2.30 (SPIHD/GPIO27)
Other:
- sheet 3V3Filter: file usb-uart.kicad_sch -> 3v3filter.kicad_sch
- sheet USB: file untitled.kicad_sch -> usb.kicad_sch
Changed lines of the file:
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@@
   )
   (no_connect (at 218.44 31.75))
+  (no_connect (at 242.062 80.772))
   (no_connect (at 242.062 113.792))
   (no_connect (at 176.022 78.232))
@@
   (no_connect (at 242.062 101.092))
   (no_connect (at 242.062 98.552))
-  (no_connect (at 242.062 96.012))
   (no_connect (at 242.062 93.472))
   (no_connect (at 242.062 70.612))
@@
     (effects (font (size 1.27 1.27)) (justify left bottom))
   )
-  (label "PDU_EN" (at 242.062 80.772 0) (fields_autoplaced)
+  (label "PDU_EN" (at 242.062 96.012 0) (fields_autoplaced)
     (effects (font (size 1.27 1.27)) (justify left bottom))
   )
@@
       (effects (font (size 1.27 1.27)) (justify left))
     )
-    (property "Footprint" "Capacitor_SMD:C_0603_1608Metric" (at 268.732 127.762 0)
+    (property "Footprint" "Capacitor_SMD:C_0402_1005Metric" (at 268.732 127.762 0)
       (effects (font (size 1.27 1.27)) hide)
     )
@@
       (effects (font (size 1.27 1.27)) (justify left))
     )
-    (property "Footprint" "Capacitor_SMD:C_0603_1608Metric" (at 270.002 139.192 0)
+    (property "Footprint" "Capacitor_SMD:C_0402_1005Metric" (at 270.002 139.192 0)
       (effects (font (size 1.27 1.27)) hide)
     )
@@
       (effects (font (size 1.27 1.27)) (justify left bottom))
     )
-    (property "Sheetfile" "usb-uart.kicad_sch" (at 78.486 88.4686 0)
+    (property "Sheetfile" "3v3filter.kicad_sch" (at 78.486 88.4686 0)
       (effects (font (size 1.27 1.27)) (justify left top))
     )
@@
       (effects (font (size 1.27 1.27)) (justify left bottom))
     )
-    (property "Sheetfile" "untitled.kicad_sch" (at 57.404 120.9806 0)
+    (property "Sheetfile" "usb.kicad_sch" (at 57.404 120.9806 0)
       (effects (font (size 1.27 1.27)) (justify left top))
     )

Commit message: 3v3logging moved to buck output
Other:
- sheet Bucks ports: added 3V3LOG; removed none
- sheet Switches+RBUS ports: added none; removed 3V3LOG
Changed lines of the file:
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@@
+    (effects (font (size 1.27 1.27)) (justify right bottom))
+  )
+  (label "3V3LOG" (at 78.74 50.546 180) (fields_autoplaced)
     (effects (font (size 1.27 1.27)) (justify right bottom))
   )
@@
   (label "DeploymentVoltage" (at 65.786 148.844 0) (fields_autoplaced)
     (effects (font (size 1.27 1.27)) (justify left bottom))
-  )
-  (label "3V3LOG" (at 35.052 84.328 180) (fields_autoplaced)
-    (effects (font (size 1.27 1.27)) (justify right bottom))
   )
   (label "SCL" (at 96.012 167.132 0) (fields_autoplaced)
@@
       (effects (font (size 1.27 1.27)) (justify left))
     )
-    (pin "3V3LOG" input (at 35.052 84.328 180)
-      (effects (font (size 1.27 1.27)) (justify left))
-    )
     (instances
       (project "Switcher"
@@
       (effects (font (size 1.27 1.27)) (justify right))
     )
-    (instances
+    (pin "3V3LOG" input (at 78.74 50.546 180)
+      (effects (font (size 1.27 1.27)) (justify left))
+    )
+    (instances

Commit message: dumbass
Connections:
- net GND: now also J7.2 (-); no longer J7.1 (+)
- net at J2.1: now also J7.1 (+); no longer J7.2 (-)
Changed lines of the file:
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@@
     (stroke (width 0) (type default))
   )
-  (wire (pts (xy 235.966 31.75) (xy 235.966 29.21))
+  (wire (pts (xy 226.06 29.21) (xy 226.06 31.75))
     (stroke (width 0) (type default))
   )
@@
     (stroke (width 0) (type default))
   )
-  (wire (pts (xy 226.06 31.75) (xy 235.966 31.75))
-    (stroke (width 0) (type default))
-  )
   (wire (pts (xy 61.468 148.844) (xy 65.786 148.844))
     (stroke (width 0) (type default))
@@
   )
   (wire (pts (xy 131.572 192.532) (xy 136.652 192.532))
+    (stroke (width 0) (type default))
+  )
+  (wire (pts (xy 233.426 29.21) (xy 226.06 29.21))
     (stroke (width 0) (type default))
   )
@@
     )
   )
-  (symbol (lib_id "power:GND") (at 233.426 29.21 0) (unit 1)
+  (symbol (lib_id "power:GND") (at 235.966 29.21 0) (unit 1)
     (in_bom yes) (on_board yes) (dnp no) (fields_autoplaced)
-    (property "Reference" "#PWR0185" (at 233.426 35.56 0)
-      (effects (font (size 1.27 1.27)) hide)
-    )
-    (property "Value" "GND" (at 233.426 33.6534 0)
-      (effects (font (size 1.27 1.27)))
-    )
-    (property "Footprint" "" (at 233.426 29.21 0)
-      (effects (font (size 1.27 1.27)) hide)
-    )
-    (property "Datasheet" "" (at 233.426 29.21 0)
-      (effects (font (size 1.27 1.27)) hide)
-    )
+    (property "Reference" "#PWR0185" (at 235.966 35.56 0)
+      (effects (font (size 1.27 1.27)) hide)
+    )
+    (property "Value" "GND" (at 235.966 33.6534 0)
+      (effects (font (size 1.27 1.27)))
+    )
+    (property "Footprint" "" (at 235.966 29.21 0)
+      (effects (font (size 1.27 1.27)) hide)
+    )
+    (property "Datasheet" "" (at 235.966 29.21 0)
+      (effects (font (size 1.27 1.27)) hide)
+    )

Commit message: new layout
Parts:
- removed J2: XT60PW-F, iclr:AMASS_XT60PW-F, symbol iclr:XT60PW-F
- added J9: XT60PW-M, iclr:AMASS_XT60PW-M, symbol iclr:XT60PW-M
Connections:
- net +12V: now also J9.1 (+)
- net at J7.1 (+): now also J9.2 (-)
- no-connect marks 31 -> 30
Changed lines of the file:
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@@
   (junction (at 136.652 192.532) (diameter 0) (color 0 0 0 0)
   )
-  (no_connect (at 218.44 31.75))
   (no_connect (at 242.062 80.772))
   (no_connect (at 242.062 113.792))
@@
   (no_connect (at 176.022 73.152))
   (no_connect (at 242.062 123.952))
+  (wire (pts (xy 233.426 29.464) (xy 233.426 29.21))
+    (stroke (width 0) (type default))
+  )
   (wire (pts (xy 129.032 170.942) (xy 122.682 170.942))
     (stroke (width 0) (type default))
@@
     (stroke (width 0) (type default))
   )
+  (wire (pts (xy 213.614 30.48) (xy 213.614 29.464))
+    (stroke (width 0) (type default))
+  )
   (wire (pts (xy 61.468 147.574) (xy 61.468 148.844))
     (stroke (width 0) (type default))
@@
     (stroke (width 0) (type default))
   )
+  (wire (pts (xy 216.154 29.464) (xy 233.426 29.464))
+    (stroke (width 0) (type default))
+  )
   (wire (pts (xy 162.052 165.862) (xy 169.672 165.862))
     (stroke (width 0) (type default))
@@
     (stroke (width 0) (type default))
   )
-  (wire (pts (xy 226.06 29.21) (xy 226.06 31.75))
-    (stroke (width 0) (type default))
-  )
   (wire (pts (xy 61.468 148.844) (xy 61.468 149.86))
     (stroke (width 0) (type default))
@@
     (stroke (width 0) (type default))
   )
+  (wire (pts (xy 207.772 30.48) (xy 213.614 30.48))
+    (stroke (width 0) (type default))
+  )
   (wire (pts (xy 164.592 22.352) (xy 164.592 27.432))
     (stroke (width 0) (type default))
@@
   )
   (wire (pts (xy 131.572 192.532) (xy 136.652 192.532))
-    (stroke (width 0) (type default))
-  )
-  (wire (pts (xy 233.426 29.21) (xy 226.06 29.21))
     (stroke (width 0) (type default))
   )
@@
     )
   )
-  (symbol (lib_id "power:+12V") (at 223.52 31.75 0) (unit 1)
-    (in_bom yes) (on_board yes) (dnp no)
-    (property "Reference" "#PWR0184" (at 223.52 35.56 0)
-      (effects (font (size 1.27 1.27)) hide)
-    )
-    (property "Value" "+12V" (at 223.52 26.67 0)
-      (effects (font (size 1.27 1.27)))
-    )
-    (property "Footprint" "" (at 223.52 31.75 0)
-      (effects (font (size 1.27 1.27)) hide)
-    )
-    (property "Datasheet" "" (at 223.52 31.75 0)
+  (symbol (lib_id "power:+12V") (at 207.772 30.48 0) (unit 1)
+    (in_bom yes) (on_board yes) (dnp no)
+    (property "Reference" "#PWR0184" (at 207.772 34.29 0)
+      (effects (font (size 1.27 1.27)) hide)
+    )
+    (property "Value" "+12V" (at 207.518 26.416 0)
+      (effects (font (size 1.27 1.27)))
+    )
+    (property "Footprint" "" (at 207.772 30.48 0)
+      (effects (font (size 1.27 1.27)) hide)
+    )
+    (property "Datasheet" "" (at 207.772 30.48 0)
       (effects (font (size 1.27 1.27)) hide)
     )
@@
     )
   )
-  (symbol (lib_id "iclr:XT60PW-F") (at 223.52 41.91 270) (unit 1)
-    (in_bom yes) (on_board yes) (dnp no) (fields_autoplaced)
-    (property "Reference" "J2" (at 229.362 41.0753 90)
-      (effects (font (size 1.27 1.27)) (justify left))
-    )
-    (property "Value" "XT60PW-F" (at 229.362 43.6122 90)
-      (effects (font (size 1.27 1.27)) (justify left))
-    )
-    (property "Footprint" "iclr:AMASS_XT60PW-F" (at 223.52 41.91 0)
-      (effects (font (size 1.27 1.27)) (justify bottom) hide)
-    )
-    (property "Datasheet" "" (at 223.52 41.91 0)
-      (effects (font (size 1.27 1.27)) hide)
-    )
-    (property "PARTREV" "V1.2" (at 223.52 41.91 0)
-      (effects (font (size 1.27 1.27)) (justify bottom) hide)
-    )
-    (property "STANDARD" "Manufacturer Recommendations" (at 223.52 41.91 0)
-      (effects (font (size 1.27 1.27)) (justify bottom) hide)
-    )
-    (property "MAXIMUM_PACKAGE_HEIGHT" "8.4 mm" (at 223.52 41.91 0)
-      (effects (font (size 1.27 1.27)) (justify bottom) hide)
-    )
-    (property "MANUFACTURER" "AMASS" (at 223.52 41.91 0)
-      (effects (font (size 1.27 1.27)) (justify bottom) hide)
-    )
-    (pin "1")
-    (pin "2")
-    (pin "S1")
-    (pin "S2")
-    (instances
-      (project "Switcher"
-        (path "/e63e39d7-6ac0-4ffd-8aa3-1841a4541b55"
-          (reference "J2") (unit 1)
-        )
-      )
-    )
-  )
   (symbol (lib_id "Device:Crystal_GND24") (at 262.382 132.842 90) (unit 1)
     (in_bom yes) (on_board yes) (dnp no)
@@
         (path "/e63e39d7-6ac0-4ffd-8aa3-1841a4541b55"
           (reference "#PWR0155") (unit 1)
+        )
+      )
+    )
+  )
+  (symbol (lib_id "iclr:XT60PW-M") (at 216.154 19.304 90) (unit 1)
+    (in_bom yes) (on_board yes) (dnp no) (fields_autoplaced)
+    (property "Reference" "J9" (at 219.456 18.6603 90)
+      (effects (font (size 1.27 1.27)) (justify right))
+    )
+    (property "Value" "XT60PW-M" (at 219.456 20.5813 90)
+      (effects (font (size 1.27 1.27)) (justify right))
+    )
+    (property "Footprint" "iclr:AMASS_XT60PW-M" (at 216.154 19.304 0)
+      (effects (font (size 1.27 1.27)) (justify bottom) hide)
+    )
+    (property "Datasheet" "" (at 216.154 19.304 0)
+      (effects (font (size 1.27 1.27)) hide)
+    )
+    (property "STANDARD" "Manufacturer recommendations" (at 216.154 19.304 0)
+      (effects (font (size 1.27 1.27)) (justify bottom) hide)
+    )
+    (property "MANUFACTURER" "AMASS" (at 216.154 19.304 0)
+      (effects (font (size 1.27 1.27)) (justify bottom) hide)
+    )
+    (property "PARTREV" "V1.2" (at 216.154 19.304 0)
+      (effects (font (size 1.27 1.27)) (justify bottom) hide)
+    )
+    (property "MAXIMUM_PACKAGE_HEIGHT" "8.4 mm" (at 216.154 19.304 0)
+      (effects (font (size 1.27 1.27)) (justify bottom) hide)
+    )
+    (pin "1")
+    (pin "2")
+    (instances
+      (project "Switcher"
+        (path "/e63e39d7-6ac0-4ffd-8aa3-1841a4541b55"
+          (reference "J9") (unit 1)
         )
       )
@@
   )
   (symbol (lib_id "power:GND") (at 235.966 29.21 0) (unit 1)
-    (in_bom yes) (on_board yes) (dnp no) (fields_autoplaced)
+    (in_bom yes) (on_board yes) (dnp no)
     (property "Reference" "#PWR0185" (at 235.966 35.56 0)
       (effects (font (size 1.27 1.27)) hide)
     )
-    (property "Value" "GND" (at 235.966 33.6534 0)
-      (effects (font (size 1.27 1.27)))
-    )
+    (property "Value" "GND" (at 240.284 31.242 0)
+      (effects (font (size 1.27 1.27)))
+    )

Commit message: new inductor, logging traces rerouted
Parts:
- C12: value 4.2pF -> DNP; footprint Capacitor_SMD:C_0603_1608Metric -> Capacitor_SMD:C_0402_1005Metric
- R8: value 47.5 -> DNP
Connections:
- net 3V3LOG: now also U2.11 (GPIO6/ADC1_CH5); no longer U2.48 (MTMS/JTAG/GPIO42)
- net DeploymentVoltage: now also U2.19 (GPIO14/ADC2_CH3); no longer U2.27 (GPIO21)
Changed lines of the file:
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@@
   (junction (at 136.652 192.532) (diameter 0) (color 0 0 0 0)
   )
+  (no_connect (at 176.022 126.492))
+  (no_connect (at 242.062 75.692))
   (no_connect (at 242.062 80.772))
   (no_connect (at 242.062 113.792))
@@
   (no_connect (at 176.022 80.772))
   (no_connect (at 176.022 83.312))
-  (no_connect (at 176.022 85.852))
   (no_connect (at 176.022 88.392))
   (no_connect (at 176.022 90.932))
@@
   (no_connect (at 176.022 101.092))
   (no_connect (at 176.022 103.632))
-  (no_connect (at 176.022 106.172))
   (no_connect (at 242.062 111.252))
   (no_connect (at 242.062 101.092))
@@
     (effects (font (size 1.27 1.27)) (justify right bottom))
   )
-  (label "DeploymentVoltage" (at 242.062 75.692 0) (fields_autoplaced)
-    (effects (font (size 1.27 1.27)) (justify left bottom))
+  (label "DeploymentVoltage" (at 176.022 106.172 180) (fields_autoplaced)
+    (effects (font (size 1.27 1.27)) (justify right bottom))
   )
   (label "CHIP_PU" (at 143.002 165.862 180) (fields_autoplaced)
@@
     (effects (font (size 1.27 1.27)) (justify left bottom))
   )
-  (label "3V3LOG" (at 176.022 126.492 180) (fields_autoplaced)
+  (label "3V3LOG" (at 176.022 85.852 180) (fields_autoplaced)
     (effects (font (size 1.27 1.27)) (justify right bottom))
   )
@@
       (effects (font (size 1.27 1.27)) (justify left))
     )
-    (property "Value" "4.2pF" (at 172.4654 60.0101 90)
-      (effects (font (size 1.27 1.27)) (justify left))
-    )
-    (property "Footprint" "Capacitor_SMD:C_0603_1608Metric" (at 172.212 62.992 0)
+    (property "Value" "DNP" (at 172.4654 60.0101 90)
+      (effects (font (size 1.27 1.27)) (justify left))
+    )
+    (property "Footprint" "Capacitor_SMD:C_0402_1005Metric" (at 172.212 62.992 0)
       (effects (font (size 1.27 1.27)) hide)
     )
@@
       (effects (font (size 1.27 1.27)))
     )
-    (property "Value" "47.5" (at 163.322 60.452 90)
-      (effects (font (size 1.27 1.27)))
-    )
+    (property "Value" "DNP" (at 163.322 60.452 90)
+      (effects (font (size 1.27 1.27)))
+    )
