File: Powerboard/Hardware/bucks.kicad_sch (KiCad schematic)
At the start: 24 parts, among them IC2 SiC437BED-T1-GE3, Q5 PXP012-30QLJ, Q6 PXP012-30QLJ, U1 LTC4412xS6, U8 LTC4412xS6

Commit message: reviewed
Parts:
- C40: footprint Capacitor_SMD:C_1206_3216Metric -> Capacitor_Tantalum_SMD:CP_EIA-7343-31_Kemet-D
- R29: value 51k -> 50k
Connections:
- net GND: now also R31.2
- net Vdd: no longer R31.2
Changed lines of the file:
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@@
+    (stroke (width 0) (type default))
+  )
+  (wire (pts (xy 183.642 101.092) (xy 185.166 101.092))
     (stroke (width 0) (type default))
   )
@@
   )
   (label "VOUT" (at 78.994 104.902 0) (fields_autoplaced)
-    (effects (font (size 1.27 1.27)) (justify left bottom))
-  )
-  (label "Vdd" (at 183.642 101.092 0) (fields_autoplaced)
     (effects (font (size 1.27 1.27)) (justify left bottom))
   )
@@
     )
   )
+  (symbol (lib_id "power:GND") (at 83.312 96.012 0) (unit 1)
+    (in_bom yes) (on_board yes) (dnp no)
+    (property "Reference" "#PWR0167" (at 83.312 102.362 0)
+      (effects (font (size 1.27 1.27)) hide)
+    )
+    (property "Value" "GND" (at 83.312 100.33 0)
+      (effects (font (size 1.27 1.27)))
+    )
+    (property "Footprint" "" (at 83.312 96.012 0)
+      (effects (font (size 1.27 1.27)) hide)
+    )
+    (property "Datasheet" "" (at 83.312 96.012 0)
+      (effects (font (size 1.27 1.27)) hide)
+    )
+    (pin "1")
+    (instances
+      (project "Switcher"
+        (path "/e63e39d7-6ac0-4ffd-8aa3-1841a4541b55/e469982c-3823-4665-9e6d-e90b00c2da09"
+          (reference "#PWR0167") (unit 1)
+        )
+      )
+    )
+  )
   (symbol (lib_id "power:GNDA") (at 155.956 138.938 0) (unit 1)
     (in_bom yes) (on_board yes) (dnp no) (fields_autoplaced)
@@
         (path "/e63e39d7-6ac0-4ffd-8aa3-1841a4541b55/e469982c-3823-4665-9e6d-e90b00c2da09"
           (reference "#PWR04") (unit 1)
+        )
+      )
+    )
+  )
+  (symbol (lib_id "power:GND") (at 198.12 109.728 0) (unit 1)
+    (in_bom yes) (on_board yes) (dnp no)
+    (property "Reference" "#PWR0111" (at 198.12 116.078 0)
+      (effects (font (size 1.27 1.27)) hide)
+    )
+    (property "Value" "GND" (at 198.12 114.046 0)
+      (effects (font (size 1.27 1.27)))
+    )
+    (property "Footprint" "" (at 198.12 109.728 0)
+      (effects (font (size 1.27 1.27)) hide)
+    )
+    (property "Datasheet" "" (at 198.12 109.728 0)
+      (effects (font (size 1.27 1.27)) hide)
+    )
+    (pin "1")
+    (instances
+      (project "Switcher"
+        (path "/e63e39d7-6ac0-4ffd-8aa3-1841a4541b55/e469982c-3823-4665-9e6d-e90b00c2da09"
+          (reference "#PWR0111") (unit 1)
         )
       )
@@
       (effects (font (size 1.27 1.27)) (justify left))
     )
-    (property "Footprint" "Capacitor_SMD:C_1206_3216Metric" (at 169.672 85.852 0)
+    (property "Footprint" "Capacitor_Tantalum_SMD:CP_EIA-7343-31_Kemet-D" (at 169.672 85.852 0)
       (effects (font (size 1.27 1.27)) hide)
     )
@@
     )
   )
-  (symbol (lib_id "power:GNDA") (at 198.12 109.728 0) (unit 1)
-    (in_bom yes) (on_board yes) (dnp no) (fields_autoplaced)
-    (property "Reference" "#PWR06" (at 198.12 116.078 0)
-      (effects (font (size 1.27 1.27)) hide)
-    )
-    (property "Value" "GNDA" (at 198.12 113.8635 0)
-      (effects (font (size 1.27 1.27)))
-    )
-    (property "Footprint" "" (at 198.12 109.728 0)
-      (effects (font (size 1.27 1.27)) hide)
-    )
-    (property "Datasheet" "" (at 198.12 109.728 0)
-      (effects (font (size 1.27 1.27)) hide)
-    )
-    (pin "1")
-    (instances
-      (project "Switcher"
-        (path "/e63e39d7-6ac0-4ffd-8aa3-1841a4541b55/e469982c-3823-4665-9e6d-e90b00c2da09"
-          (reference "#PWR06") (unit 1)
-        )
-      )
-    )
-  )
   (symbol (lib_id "Device:C_Small") (at 58.674 114.808 180) (unit 1)
     (in_bom yes) (on_board yes) (dnp no)
@@
     )
   )
-  (symbol (lib_id "power:GNDA") (at 83.312 96.012 0) (unit 1)
-    (in_bom yes) (on_board yes) (dnp no) (fields_autoplaced)
-    (property "Reference" "#PWR08" (at 83.312 102.362 0)
-      (effects (font (size 1.27 1.27)) hide)
-    )
-    (property "Value" "GNDA" (at 83.312 100.1475 0)
-      (effects (font (size 1.27 1.27)))
-    )
-    (property "Footprint" "" (at 83.312 96.012 0)
-      (effects (font (size 1.27 1.27)) hide)
-    )
-    (property "Datasheet" "" (at 83.312 96.012 0)
-      (effects (font (size 1.27 1.27)) hide)
-    )
-    (pin "1")
-    (instances
-      (project "Switcher"
-        (path "/e63e39d7-6ac0-4ffd-8aa3-1841a4541b55/e469982c-3823-4665-9e6d-e90b00c2da09"
-          (reference "#PWR08") (unit 1)
-        )
-      )
-    )
-  )
   (symbol (lib_id "power:GND") (at 181.864 88.392 0) (unit 1)
     (in_bom yes) (on_board yes) (dnp no)
@@
     )
   )
+  (symbol (lib_id "power:GND") (at 185.166 101.092 0) (unit 1)
+    (in_bom yes) (on_board yes) (dnp no)
+    (property "Reference" "#PWR0106" (at 185.166 107.442 0)
+      (effects (font (size 1.27 1.27)) hide)
+    )
+    (property "Value" "GND" (at 185.166 105.41 0)
+      (effects (font (size 1.27 1.27)))
+    )
+    (property "Footprint" "" (at 185.166 101.092 0)
+      (effects (font (size 1.27 1.27)) hide)
+    )
+    (property "Datasheet" "" (at 185.166 101.092 0)
+      (effects (font (size 1.27 1.27)) hide)
+    )
+    (pin "1")
+    (instances
+      (project "Switcher"
+        (path "/e63e39d7-6ac0-4ffd-8aa3-1841a4541b55/e469982c-3823-4665-9e6d-e90b00c2da09"
+          (reference "#PWR0106") (unit 1)
+        )
+      )
+    )
+  )
   (symbol (lib_id "power:GND") (at 159.512 124.968 0) (unit 1)
     (in_bom yes) (on_board yes) (dnp no) (fields_autoplaced)
@@
   (symbol (lib_id "Device:R_Small") (at 180.086 110.998 0) (unit 1)
     (in_bom yes) (on_board yes) (dnp no) (fields_autoplaced)
-    (property "Reference" "R29" (at 181.5846 110.3543 0)
+    (property "Reference" "R29" (at 181.5846 110.1633 0)
       (effects (font (size 1.27 1.27)) (justify left))
     )
-    (property "Value" "51k" (at 181.5846 112.2753 0)
+    (property "Value" "50k" (at 181.5846 112.7002 0)
       (effects (font (size 1.27 1.27)) (justify left))
     )
