File: Powerboard/Hardware/Switcher.kicad_pcb (KiCad board)
At the start: 4 copper layers, 47 x 50 mm, 118 parts, among them IC2 SiC437BED-T1-GE3, J1 Conn_01x03_MountingPin, J2 XT60PW-F, J3 USB_C_Receptacle_USB2.0, J4 Conn_01x02_Male, J5 Conn_01x08_Male, J6 Conn_01x02_Male, J7 XT60PW-M, J8 Conn_01x04_Male, Q1 PXP012-30QLJ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

Commit message: update
Parts:
- moved Q3 0.56 mm to (99.9, 35.8)
Routing:
- net Net-(Q5-G): track 5.57 -> 4.10 mm
- net +12V: track 21.9 -> 21.0 mm, vias 11 -> 20
- net Net-(J5-Pin_5): track 6.83 -> 6.13 mm, vias 23 -> 17
- net Net-(Q3-G): track 10.5 -> 11.0 mm
- net VBUS: vias 5 -> 4
- net Net-(Q3-S_1): vias 4 -> 8
- net Net-(Q1-S_1): vias 3 -> 4
- net Net-(J5-Pin_4): vias 7 -> 9
- net GND: vias 109 -> 108

Commit message: nothing
Routing:
- net GND: vias 108 -> 107
Changed lines of the file:
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@@
   (via (at 112.9 37.388888) (size 0.6) (drill 0.3) (layers "F.Cu" "B.Cu") (free) (net 3))
   (via (at 86.749998 23.6) (size 0.6) (drill 0.3) (layers "F.Cu" "B.Cu") (free) (net 3))
-  (via (at 96 54.5) (size 0.6) (drill 0.3) (layers "F.Cu" "B.Cu") (free) (net 3))
   (via (at 74.27 72.26) (size 0.6) (drill 0.3) (layers "F.Cu" "B.Cu") (free) (net 3))
   (via (at 93.5 47.7) (size 0.8) (drill 0.4) (layers "F.Cu" "B.Cu") (net 3))
@@
   (segment (start 89.79 54.86) (end 89.365 54.86) (width 0.2) (layer "F.Cu") (net 46))
   (segment (start 87.425 57.46) (end 87 57.46) (width 0.2) (layer "F.Cu") (net 46))
-  (segment (start 85.012 59.448) (end 87 57.46) (width 0.2) (layer "F.Cu") (net 46))
-  (segment (start 84.322 59.448) (end 85.012 59.448) (width 0.2) (layer "F.Cu") (net 46))
-  (segment (start 84.1 60.3375) (end 84.1 59.67) (width 0.2) (layer "F.Cu") (net 46))
-  (segment (start 84.1 59.67) (end 84.322 59.448) (width 0.2) (layer "F.Cu") (net 46))
+  (segment (start 85.46 59) (end 87 57.46) (width 0.2) (layer "F.Cu") (net 46))
+  (segment (start 84.9 59) (end 85.46 59) (width 0.2) (layer "F.Cu") (net 46))
+  (segment (start 84.1 59.8) (end 84.9 59) (width 0.2) (layer "F.Cu") (net 46))
+  (segment (start 84.1 60.3375) (end 84.1 59.8) (width 0.2) (layer "F.Cu") (net 46))
   (via (at 89.79 54.86) (size 0.45) (drill 0.3) (layers "F.Cu" "B.Cu") (net 46))
   (via (at 87 57.46) (size 0.45) (drill 0.3) (layers "F.Cu" "B.Cu") (net 46))
@@
     (polygon
       (pts
-        (xy 98.3 50.7)
+        (xy 98.3 49.9)
         (xy 98.3 53.4)
         (xy 94.7 53.4)
@@
         (xy 87 48.8)
         (xy 91.3 48.8)
-        (xy 94.44 53.55)
-        (xy 98.4 59)
+        (xy 94.5 53.7)
+        (xy 98.4 53.7)
         (xy 98.4 62)
-        (xy 90.5 62)
+        (xy 90.1 61.9)
         (xy 89.8 54.3)
         (xy 87 54.3)

Commit message: nothing
Parts:
- moved R4 0.84 mm to (73.9, 43.1)
- moved D2 0.57 mm to (70.6, 54.4)
- moved TP4 0.55 mm to (75.9, 49.8)
- moved C52 0.26 mm to (77.8, 49.5)
- moved C51 0.23 mm to (77.7, 48.5)
- moved R15 0.15 mm to (74.1, 49.5), turned to 90 degrees
- moved C20 0.15 mm to (74.1, 51.9), turned to -90 degrees
- moved R16 0.13 mm to (72.1, 51.8)
- moved TP5 0.12 mm to (68.2, 35.3)
- moved TXLED1 0.12 mm to (75.4, 52.3)
- moved R17 0.12 mm to (69.2, 51.8)
- moved R23 0.11 mm to (68.4, 53.4)
- moved R5 0.11 mm to (76.3, 52.3)
- moved L2 0.07 mm to (75.7, 43.2)
- moved C14 0.07 mm to (76.2, 44.6)
Connections:
- C49 pad 2: /3V3Filter/GNDA -> GND
- R1 pad 2: /3V3Filter/GNDA -> GND
- U4 pad 4: /3V3Filter/GNDA -> GND
Routing:
- net /3V3Filter/GNDA: vias 1 -> 0
- removed copper zone on F.Cu, net /3V3Filter/GNDA
