File: Powerboard/Hardware/PDU.kicad_pcb (KiCad board)
At the start: 4 copper layers, 60 x 50 mm, 118 parts, among them IC2 SiC437BED-T1-GE3, J1 Conn_01x03_MountingPin, J3 USB_C_Receptacle_USB2.0, J4 Conn_01x02_Male, J5 Conn_01x08_Male, J6 Conn_01x02_Male, J7 XT60PW-M, J8 Conn_01x04_Male, J9 XT60PW-M, Q1 PXP012-30QLJ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

Commit message: added some commands, hardware fixes
Parts:
- removed 12VLED1: 12V_LED, Resistor_SMD:R_0402_1005Metric
- added BATTLED1: BATT_LED, LED_SMD:LED_0402_1005Metric, F.Cu at (121.6, 35.7)
- added DEPLED1: DEP_LED, LED_SMD:LED_0402_1005Metric, F.Cu at (123.0, 42.5)
- added LOGICLED1: LOGIC_LED, LED_SMD:LED_0402_1005Metric, F.Cu at (121.4, 40.2)
- added R27: 3k, Resistor_SMD:R_0402_1005Metric, F.Cu at (122.0, 41.6)
- added R28: 47k, Resistor_SMD:R_0402_1005Metric, F.Cu at (122.0, 43.5)
- added R32: 10k, Resistor_SMD:R_0402_1005Metric, F.Cu at (123.1, 44.4)
- added R33: 470, Resistor_SMD:R_0402_1005Metric, F.Cu at (120.4, 39.3)
- 3V3LED1, TXLED1: footprint Resistor_SMD:R_0402_1005Metric -> LED_SMD:LED_0402_1005Metric
- R10, R11: moved to F.Cu
- moved TP1 6.69 mm to (78.2, 32.3)
- moved R11 6.41 mm to (75.2, 27.7)
- moved R10 6.40 mm to (76.1, 27.7)
- moved R12 3.54 mm to (88.1, 36.1), turned to 180 degrees
- moved R9 2.59 mm to (120.5, 34.8)
- moved USBLED1 2.57 mm to (87.1, 37.0), turned to 0 degrees
- moved D1 1.22 mm to (73.7, 30.6), turned to -45 degrees
- moved J3 1.01 mm to (82.3, 27.3)
- moved C24 0.74 mm to (114.8, 52.3)
- moved TP2 0.36 mm to (71.4, 32.2)
- moved C11 0.18 mm to (75.1, 32.8)
- moved R7 0.18 mm to (120.5, 37.1)
- moved 3V3LED1 0.17 mm to (121.5, 38.0)
Connections:
- net /12V_SWITCH renamed /DEP_SWITCH
- net /3V3LOG renamed /LogicVoltage
- net /3V3_SWITCH renamed /LOGIC_SWITCH
- net /DeploymentVoltage renamed /BattVoltage
- net /PDU_EN renamed /ARMING
- D1 pad 3: /Data+ -> /Data-
- D1 pad 4: /Data- -> /Data+
- J3 pad A6: /Data- -> /Data+
- J3 pad A7: /Data+ -> /Data-
- J3 pad B6: /Data- -> /Data+
- J3 pad B7: /Data+ -> /Data-
- TP1 pad 1: /Data+ -> /Data-
- TP2 pad 1: /Data- -> /Data+
- U2 pad 18: unconnected-(U2-GPIO13/ADC2_CH2-Pad18) -> /DepVoltage
Routing:
- net /DepVoltage: track 0.00 -> 70.9 mm, vias 0 -> 2
- net Net-(J5-Pin_4): track 9.77 -> 57.8 mm, vias 0 -> 1
- net VBUS: track 4.02 -> 16.8 mm
- net Net-(J3-CC1): track 2.58 -> 11.4 mm, vias 1 -> 2
- net /Data-: track 20.0 -> 14.0 mm, vias 2 -> 0
- net Net-(J3-CC2): track 2.44 -> 7.39 mm, vias 1 -> 2
- net /Data+: track 20.6 -> 16.6 mm
- net /BattVoltage: track 56.1 -> 57.2 mm
- net Net-(DEPLED1-A): track 0.00 -> 0.95 mm
- net GND: track 4.99 -> 4.04 mm, vias 113 -> 115
- net Net-(LOGICLED1-A): track 0.00 -> 0.95 mm
- net +3V3: track 9.18 -> 8.66 mm
- net Net-(J5-Pin_5): vias 44 -> 39
Other:
- board text added: "BATT LED"
- board text added: "DEP LED"
- board text added: "DEP SWITCH"
- board text added: "LOGIC LED"
- board text added: "LOGIC SWITCH"
- board text removed: "-"
- board text removed: "12V LED"
- board text removed: "12V SWITCH"
- board text removed: "3V3 SWITCH"

Commit message: firmware updates
Parts:
- removed Q1, Q2, Q3, Q4: PXP012-30QLJ, iclr:PXP01230QLJ
- added J2: FAN, Connector_PinHeader_2.54mm:PinHeader_1x02_P2.54mm_Vertical, F.Cu at (124.7, 60.4)
- added Q10: SQS141ELNW-T1_GE3, iclr:SQS850ENT1_GE3, F.Cu at (115.2, 41.5)
- added Q7: SQS141ELNW-T1_GE3, iclr:SQS850ENT1_GE3, F.Cu at (98.3, 61.3)
- added Q8: SQS141ELNW-T1_GE3, iclr:SQS850ENT1_GE3, F.Cu at (98.3, 67.2)
- added Q9: SQS141ELNW-T1_GE3, iclr:SQS850ENT1_GE3, F.Cu at (115.1, 35.6)
- R31: value 200k -> 100k
- moved R11 0.55 mm to (75.6, 28.0)
- moved R10 0.52 mm to (76.5, 28.0)
Routing:
- net Net-(J6-Pin_1): track 50.2 -> 55.5 mm
- net /LIPOPOWER: track 41.9 -> 40.9 mm
- net Net-(Q10-G): track 14.5 -> 15.4 mm
- net Net-(Q7-G): track 14.9 -> 15.7 mm
- net Net-(J5-Pin_4): track 57.8 -> 58.6 mm, vias 1 -> 17
- net VBUS: track 16.8 -> 16.1 mm
- net Net-(J3-CC2): track 7.39 -> 6.86 mm
- net Net-(J3-CC1): track 11.4 -> 10.9 mm
- net RBUS_uC_V: vias 2 -> 18
- net Net-(Q7-S_1): vias 0 -> 12
- net Net-(Q3-S_1): vias 10 -> 0
- net Net-(Q10-S_1): vias 0 -> 12
- net Net-(J7-+): vias 16 -> 10
- net Net-(J5-Pin_5): vias 39 -> 29
- net GND: vias 115 -> 113
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- added copper zone on B.Cu, net Net-(J5-Pin_4)
- added copper zone on B.Cu, net Net-(Q10-S_1)
- added copper zone on F.Cu, net Net-(Q10-S_1)
- added copper zone on B.Cu, net Net-(Q7-S_1)
- added copper zone on F.Cu, net Net-(Q7-S_1)
- added copper zone on B.Cu, net RBUS_uC_V
- removed copper zone on F.Cu, net Net-(Q1-S_1)
- removed copper zone on B.Cu, net Net-(Q3-S_1)
- removed copper zone on F.Cu, net Net-(Q3-S_1)
Other:
- board text added: "FAN"

Commit message: v2.1
Parts:
- removed JP3: SolderJumper_2_Bridged, Jumper:SolderJumper-2_P1.3mm_Bridged_RoundedPad1.0x1.5mm
- removed R19: 10k, Resistor_SMD:R_0402_1005Metric
- added JP1: SolderJumper_2_Bridged, Jumper:SolderJumper-2_P1.3mm_Bridged_RoundedPad1.0x1.5mm, F.Cu at (71.4, 60.4)
- added Q1: SSM3K15AMFV,L3F, Package_TO_SOT_SMD:SOT-723, F.Cu at (110.3, 45.6)
- added R34: 1k, Resistor_SMD:R_0402_1005Metric, F.Cu at (109.0, 45.6)
- added R35: 10k, Resistor_SMD:R_0402_1005Metric, F.Cu at (111.7, 45.6)
- moved J2 50.4 mm to (74.9, 68.6)
- moved R4 0.67 mm to (73.8, 44.9)
- moved C10 0.45 mm to (73.2, 42.5)
- moved R31 0.42 mm to (104.5, 38.5)
- moved R29 0.40 mm to (103.6, 38.5)
- moved C18 0.25 mm to (78.8, 57.4)
- moved C19 0.25 mm to (77.0, 57.4)
- moved C20 0.25 mm to (81.0, 67.7)
- moved R15 0.25 mm to (82.0, 63.8)
- moved R16 0.25 mm to (80.0, 66.0)
- moved R17 0.25 mm to (77.0, 66.0)
- moved R23 0.25 mm to (75.4, 63.3)
- moved U5 0.25 mm to (78.5, 61.6)
- moved D2 0.25 mm to (78.5, 68.7)
- moved LOGICLED1 0.07 mm to (121.5, 40.2)
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Connections:
- J6 pad 2: GND -> +3V3
- Q9 pad 7: unconnected-(Q9-D_3-Pad7) -> +12V
- U7 pad 3: Net-(J6-Pin_1) -> /Switches+RBUS/CTL
Routing:
- net Net-(J6-Pin_1): track 55.5 -> 50.6 mm
- net +12V: track 8.85 -> 13.2 mm
- net /CAN_TX: track 23.2 -> 26.7 mm, vias 2 -> 0
- net /Switches+RBUS/CTL: track 0.00 -> 3.31 mm
- net +3V3: track 8.66 -> 6.51 mm, vias 11 -> 10
- net Net-(IC2-EN): track 9.63 -> 11.6 mm, vias 17 -> 15
- net Net-(J5-Pin_4): track 58.6 -> 56.6 mm, vias 17 -> 21
- net /TXD: track 8.17 -> 7.45 mm
- net Net-(U2-U0TXD/PROG/GPIO43): track 3.35 -> 3.92 mm
- net /CAN_RX: track 20.3 -> 20.7 mm, vias 2 -> 0
- net RBUS_uC_V: track 20.1 -> 19.8 mm, vias 18 -> 21
- net Net-(J5-Pin_5): vias 29 -> 28
Other:
- board text added: "Lightning McQueen v2.1"
- board text removed: "Lightning McQueen v2.0"

Commit message: hardware update
Parts:
- moved G*** 3.46 mm to (83.1, 62.9)
- moved R10 3.00 mm to (73.8, 26.9)
- moved J3 2.46 mm to (79.8, 27.5)
- moved locked 2.23 mm to (103.8, 47.3)
- moved R11 1.98 mm to (73.8, 28.8), turned to 90 degrees
- moved TP2 1.44 mm to (70.0, 32.1)
- moved D1 1.44 mm to (72.6, 31.6), turned to 0 degrees
- moved C11 1.08 mm to (76.2, 32.8), turned to 0 degrees
- moved G*** 0.99 mm to (79.0, 36.2)
- moved USBLED1 0.66 mm to (86.7, 37.5), turned to 90 degrees
- moved R12 0.65 mm to (87.6, 36.5), turned to -90 degrees
- moved TP1 0.08 mm to (78.1, 32.2)
Routing:
- net /Data-: track 13.9 -> 9.30 mm
- net /DepVoltage: track 70.9 -> 74.0 mm
- net /BattVoltage: track 56.7 -> 59.8 mm
- net /Data+: track 16.5 -> 14.2 mm
- net Net-(J3-CC1): track 10.9 -> 8.74 mm
- net VBUS: track 16.1 -> 14.6 mm
- net Net-(J6-Pin_1): track 50.6 -> 49.5 mm
- net Net-(J4-Pin_1): track 41.2 -> 40.4 mm
