File: Powerboard/Hardware/3v3bucks.kicad_sch (KiCad schematic)
At the start: 26 parts, among them IC2 SiC437BED-T1-GE3, Q5 PXP012-30QLJ, Q6 PXP012-30QLJ, U1 LTC4412xS6, U8 LTC4412xS6

Commit message: firmware updates
Parts:
- R31: value 200k -> 100k
Changed lines of the file:
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@@
     (pin "2")
     (instances
-      (project "Switcher"
+      (project "PDU"
         (path "/e63e39d7-6ac0-4ffd-8aa3-1841a4541b55/e469982c-3823-4665-9e6d-e90b00c2da09"
           (reference "C44") (unit 1)
@@
     (pin "1")
     (instances
-      (project "Switcher"
+      (project "PDU"
         (path "/e63e39d7-6ac0-4ffd-8aa3-1841a4541b55/e469982c-3823-4665-9e6d-e90b00c2da09"
           (reference "#PWR04") (unit 1)
@@
     (pin "2")
     (instances
-      (project "Switcher"
+      (project "PDU"
         (path "/e63e39d7-6ac0-4ffd-8aa3-1841a4541b55/e469982c-3823-4665-9e6d-e90b00c2da09"
           (reference "C42") (unit 1)
@@
     (pin "2")
     (instances
-      (project "Switcher"
+      (project "PDU"
         (path "/e63e39d7-6ac0-4ffd-8aa3-1841a4541b55/e469982c-3823-4665-9e6d-e90b00c2da09"
           (reference "R30") (unit 1)
@@
     (pin "1")
     (instances
-      (project "Switcher"
+      (project "PDU"
         (path "/e63e39d7-6ac0-4ffd-8aa3-1841a4541b55/e469982c-3823-4665-9e6d-e90b00c2da09"
           (reference "#PWR0149") (unit 1)
@@
     (pin "2")
     (instances
-      (project "Switcher"
+      (project "PDU"
         (path "/e63e39d7-6ac0-4ffd-8aa3-1841a4541b55/e469982c-3823-4665-9e6d-e90b00c2da09"
           (reference "C30") (unit 1)
@@
     (pin "2")
     (instances
-      (project "Switcher"
+      (project "PDU"
         (path "/e63e39d7-6ac0-4ffd-8aa3-1841a4541b55/e469982c-3823-4665-9e6d-e90b00c2da09"
           (reference "R21") (unit 1)
@@
     (pin "2")
     (instances
-      (project "Switcher"
+      (project "PDU"
         (path "/e63e39d7-6ac0-4ffd-8aa3-1841a4541b55/e469982c-3823-4665-9e6d-e90b00c2da09"
           (reference "C40") (unit 1)
@@
     (pin "2")
     (instances
-      (project "Switcher"
+      (project "PDU"
         (path "/e63e39d7-6ac0-4ffd-8aa3-1841a4541b55/e469982c-3823-4665-9e6d-e90b00c2da09"
           (reference "L3") (unit 1)
@@
     (pin "1")
     (instances
-      (project "Switcher"
+      (project "PDU"
         (path "/e63e39d7-6ac0-4ffd-8aa3-1841a4541b55/133f56f4-a29c-4cbf-87b7-9d99a292e3c0"
           (reference "#PWR01") (unit 1)
@@
       (effects (font (size 1.27 1.27)) (justify left))
     )
-    (property "Value" "200k" (at 183.134 98.552 90)
+    (property "Value" "100k" (at 183.134 98.552 90)
       (effects (font (size 1.27 1.27)) (justify left))
     )
@@
     (pin "2")
     (instances
-      (project "Switcher"
+      (project "PDU"
         (path "/e63e39d7-6ac0-4ffd-8aa3-1841a4541b55/e469982c-3823-4665-9e6d-e90b00c2da09"
           (reference "R31") (unit 1)
@@
     (pin "2")
     (instances
-      (project "Switcher"
+      (project "PDU"
         (path "/e63e39d7-6ac0-4ffd-8aa3-1841a4541b55/e469982c-3823-4665-9e6d-e90b00c2da09"
           (reference "C47") (unit 1)
@@
     (pin "2")
     (instances
-      (project "Switcher"
+      (project "PDU"
         (path "/e63e39d7-6ac0-4ffd-8aa3-1841a4541b55/e469982c-3823-4665-9e6d-e90b00c2da09"
           (reference "R20") (unit 1)
@@
     (pin "9")
     (instances
-      (project "Switcher"
+      (project "PDU"
         (path "/e63e39d7-6ac0-4ffd-8aa3-1841a4541b55/e469982c-3823-4665-9e6d-e90b00c2da09"
           (reference "IC2") (unit 1)
@@
     (pin "2")
     (instances
-      (project "Switcher"
+      (project "PDU"
         (path "/e63e39d7-6ac0-4ffd-8aa3-1841a4541b55/e469982c-3823-4665-9e6d-e90b00c2da09"
           (reference "C32") (unit 1)
@@
     (pin "9")
     (instances
-      (project "Switcher"
+      (project "PDU"
         (path "/e63e39d7-6ac0-4ffd-8aa3-1841a4541b55/e469982c-3823-4665-9e6d-e90b00c2da09"
           (reference "Q5") (unit 1)
@@
     (pin "2")
     (instances
-      (project "Switcher"
+      (project "PDU"
         (path "/e63e39d7-6ac0-4ffd-8aa3-1841a4541b55/e469982c-3823-4665-9e6d-e90b00c2da09"
           (reference "C46") (unit 1)
@@
     (pin "2")
     (instances
-      (project "Switcher"
+      (project "PDU"
         (path "/e63e39d7-6ac0-4ffd-8aa3-1841a4541b55/133f56f4-a29c-4cbf-87b7-9d99a292e3c0"
           (reference "R26") (unit 1)
@@
     (pin "2")
     (instances
-      (project "Switcher"
+      (project "PDU"
         (path "/e63e39d7-6ac0-4ffd-8aa3-1841a4541b55/e469982c-3823-4665-9e6d-e90b00c2da09"
           (reference "C25") (unit 1)
@@
     (pin "1")
     (instances
-      (project "Switcher"
+      (project "PDU"
         (path "/e63e39d7-6ac0-4ffd-8aa3-1841a4541b55/e469982c-3823-4665-9e6d-e90b00c2da09"
           (reference "#PWR0169") (unit 1)
@@
     (pin "9")
     (instances
-      (project "Switcher"
+      (project "PDU"
         (path "/e63e39d7-6ac0-4ffd-8aa3-1841a4541b55/e469982c-3823-4665-9e6d-e90b00c2da09"
           (reference "Q6") (unit 1)
@@
     (pin "2")
     (instances
-      (project "Switcher"
+      (project "PDU"
         (path "/e63e39d7-6ac0-4ffd-8aa3-1841a4541b55/133f56f4-a29c-4cbf-87b7-9d99a292e3c0"
           (reference "R24") (unit 1)
@@
     (pin "6")
     (instances
-      (project "Switcher"
+      (project "PDU"
         (path "/e63e39d7-6ac0-4ffd-8aa3-1841a4541b55/e469982c-3823-4665-9e6d-e90b00c2da09"
           (reference "U1") (unit 1)
@@
     (pin "1")
     (instances
-      (project "Switcher"
+      (project "PDU"
         (path "/e63e39d7-6ac0-4ffd-8aa3-1841a4541b55/e469982c-3823-4665-9e6d-e90b00c2da09"
           (reference "#PWR0183") (unit 1)
@@
     (pin "1")
     (instances
-      (project "Switcher"
+      (project "PDU"
         (path "/e63e39d7-6ac0-4ffd-8aa3-1841a4541b55/e469982c-3823-4665-9e6d-e90b00c2da09"
           (reference "#PWR0181") (unit 1)
@@
     (pin "2")
     (instances
-      (project "Switcher"
+      (project "PDU"
         (path "/e63e39d7-6ac0-4ffd-8aa3-1841a4541b55/e469982c-3823-4665-9e6d-e90b00c2da09"
           (reference "C38") (unit 1)
@@
     (pin "1")
     (instances
-      (project "Switcher"
+      (project "PDU"
         (path "/e63e39d7-6ac0-4ffd-8aa3-1841a4541b55/e469982c-3823-4665-9e6d-e90b00c2da09"
           (reference "#PWR06") (unit 1)
@@
     (pin "2")
     (instances
-      (project "Switcher"
+      (project "PDU"
         (path "/e63e39d7-6ac0-4ffd-8aa3-1841a4541b55/e469982c-3823-4665-9e6d-e90b00c2da09"
           (reference "R25") (unit 1)
@@
     (pin "1")
     (instances
-      (project "Switcher"
+      (project "PDU"
         (path "/e63e39d7-6ac0-4ffd-8aa3-1841a4541b55/e469982c-3823-4665-9e6d-e90b00c2da09"
           (reference "#PWR05") (unit 1)
@@
     (pin "1")
     (instances
-      (project "Switcher"
+      (project "PDU"
         (path "/e63e39d7-6ac0-4ffd-8aa3-1841a4541b55/e469982c-3823-4665-9e6d-e90b00c2da09"
           (reference "#PWR02") (unit 1)
@@
     (pin "2")
     (instances
-      (project "Switcher"
+      (project "PDU"
         (path "/e63e39d7-6ac0-4ffd-8aa3-1841a4541b55/e469982c-3823-4665-9e6d-e90b00c2da09"
           (reference "C15") (unit 1)
@@
     (pin "1")
     (instances
-      (project "Switcher"
+      (project "PDU"
         (path "/e63e39d7-6ac0-4ffd-8aa3-1841a4541b55/e469982c-3823-4665-9e6d-e90b00c2da09"
           (reference "#PWR0180") (unit 1)
@@
     (pin "1")
     (instances
-      (project "Switcher"
+      (project "PDU"
         (path "/e63e39d7-6ac0-4ffd-8aa3-1841a4541b55/e469982c-3823-4665-9e6d-e90b00c2da09"
           (reference "#PWR03") (unit 1)
@@
     (pin "6")
     (instances
-      (project "Switcher"
+      (project "PDU"
         (path "/e63e39d7-6ac0-4ffd-8aa3-1841a4541b55/e469982c-3823-4665-9e6d-e90b00c2da09"
           (reference "U8") (unit 1)
@@
     (pin "1")
     (instances
-      (project "Switcher"
+      (project "PDU"
         (path "/e63e39d7-6ac0-4ffd-8aa3-1841a4541b55/e469982c-3823-4665-9e6d-e90b00c2da09"
           (reference "#PWR08") (unit 1)
@@
     (pin "1")
     (instances
-      (project "Switcher"
+      (project "PDU"
         (path "/e63e39d7-6ac0-4ffd-8aa3-1841a4541b55/e469982c-3823-4665-9e6d-e90b00c2da09"
           (reference "#PWR0168") (unit 1)
@@
     (pin "1")
     (instances
-      (project "Switcher"
+      (project "PDU"
         (path "/e63e39d7-6ac0-4ffd-8aa3-1841a4541b55/e469982c-3823-4665-9e6d-e90b00c2da09"
           (reference "#PWR0166") (unit 1)
@@
     (pin "1")
     (instances
-      (project "Switcher"
+      (project "PDU"
         (path "/e63e39d7-6ac0-4ffd-8aa3-1841a4541b55/e469982c-3823-4665-9e6d-e90b00c2da09"
           (reference "#PWR0158") (unit 1)
@@
     (pin "2")
     (instances
-      (project "Switcher"
+      (project "PDU"
         (path "/e63e39d7-6ac0-4ffd-8aa3-1841a4541b55/e469982c-3823-4665-9e6d-e90b00c2da09"
           (reference "C34") (unit 1)
@@
     (pin "2")
     (instances
-      (project "Switcher"
+      (project "PDU"
         (path "/e63e39d7-6ac0-4ffd-8aa3-1841a4541b55/e469982c-3823-4665-9e6d-e90b00c2da09"
           (reference "C36") (unit 1)
@@
     (pin "1")
     (instances
-      (project "Switcher"
+      (project "PDU"
         (path "/e63e39d7-6ac0-4ffd-8aa3-1841a4541b55/e469982c-3823-4665-9e6d-e90b00c2da09"
           (reference "#PWR0150") (unit 1)
@@
     (pin "2")
     (instances
-      (project "Switcher"
+      (project "PDU"
         (path "/e63e39d7-6ac0-4ffd-8aa3-1841a4541b55/e469982c-3823-4665-9e6d-e90b00c2da09"
           (reference "R29") (unit 1)

Commit message: v2.1 ordering
Parts:
- IC2: value SiC437BED-T1-GE3 -> SiC437AED-T1-GE3
Changed lines of the file:
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@@
   (symbol (lib_id "iclr:SiC437BED-T1-GE3") (at 115.316 91.948 0) (unit 1)
     (in_bom yes) (on_board yes) (dnp no) (fields_autoplaced)
-    (property "Reference" "IC2" (at 133.096 85.759 0)
+    (property "Reference" "IC2" (at 133.096 85.09 0)
       (effects (font (size 1.27 1.27)))
     )
-    (property "Value" "SiC437BED-T1-GE3" (at 133.096 88.2959 0)
+    (property "Value" "SiC437AED-T1-GE3" (at 133.096 87.63 0)
       (effects (font (size 1.27 1.27)))
     )

Commit message: added RC snubber
Parts:
- added C16: 680pF, Capacitor_SMD:C_0603_1608Metric, symbol Device:C_Small
- added R37: 5.1, Resistor_SMD:R_0603_1608Metric, symbol Device:R_Small
Connections:
- net GND: now also R37.2
- net SW: now also C16.1
- new net: C16.2, R37.1
Changed lines of the file:
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@@
     (effects (font (size 1.27 1.27)) (justify right bottom))
+  )
+  (label "SW" (at 195.58 120.65 0) (fields_autoplaced)
+    (effects (font (size 1.27 1.27)) (justify left bottom))
   )
   (label "Vdd" (at 173.736 107.95 180) (fields_autoplaced)
@@
     )
   )
+  (symbol (lib_id "Device:R_Small") (at 195.58 128.27 0) (unit 1)
+    (in_bom yes) (on_board yes) (dnp no) (fields_autoplaced)
+    (property "Reference" "R37" (at 198.12 127.635 0)
+      (effects (font (size 1.27 1.27)) (justify left))
+    )
+    (property "Value" "5.1" (at 198.12 130.175 0)
+      (effects (font (size 1.27 1.27)) (justify left))
+    )
+    (property "Footprint" "Resistor_SMD:R_0603_1608Metric" (at 195.58 128.27 0)
+      (effects (font (size 1.27 1.27)) hide)
+    )
+    (property "Datasheet" "~" (at 195.58 128.27 0)
+      (effects (font (size 1.27 1.27)) hide)
+    )
+    (pin "1")
+    (pin "2")
+    (instances
+      (project "PDU"
+        (path "/e63e39d7-6ac0-4ffd-8aa3-1841a4541b55/e469982c-3823-4665-9e6d-e90b00c2da09"
+          (reference "R37") (unit 1)
+        )
+      )
+    )
+  )
   (symbol (lib_id "Device:R_Small") (at 29.21 117.856 0) (unit 1)
     (in_bom yes) (on_board yes) (dnp no) (fields_autoplaced)
@@
         (path "/e63e39d7-6ac0-4ffd-8aa3-1841a4541b55/e469982c-3823-4665-9e6d-e90b00c2da09"
           (reference "R24") (unit 1)
+        )
+      )
+    )
+  )
+  (symbol (lib_id "power:GND") (at 195.58 130.81 0) (unit 1)
+    (in_bom yes) (on_board yes) (dnp no) (fields_autoplaced)
+    (property "Reference" "#PWR017" (at 195.58 137.16 0)
+      (effects (font (size 1.27 1.27)) hide)
+    )
+    (property "Value" "GND" (at 195.58 135.2534 0)
+      (effects (font (size 1.27 1.27)))
+    )
+    (property "Footprint" "" (at 195.58 130.81 0)
+      (effects (font (size 1.27 1.27)) hide)
+    )
+    (property "Datasheet" "" (at 195.58 130.81 0)
+      (effects (font (size 1.27 1.27)) hide)
+    )
+    (pin "1")
+    (instances
+      (project "PDU"
+        (path "/e63e39d7-6ac0-4ffd-8aa3-1841a4541b55/e469982c-3823-4665-9e6d-e90b00c2da09"
+          (reference "#PWR017") (unit 1)
         )
       )
@@
         )
       )
+    )
+  )
+  (symbol (lib_id "Device:C_Small") (at 195.58 123.19 0) (unit 1)
+    (in_bom yes) (on_board yes) (dnp no) (fields_autoplaced)
+    (property "Reference" "C16" (at 198.12 122.5613 0)
+      (effects (font (size 1.27 1.27)) (justify left))
+    )
+    (property "Value" "680pF" (at 198.12 125.1013 0)
+      (effects (font (size 1.27 1.27)) (justify left))
+    )
+    (property "Footprint" "Capacitor_SMD:C_0603_1608Metric" (at 195.58 123.19 0)
+      (effects (font (size 1.27 1.27)) hide)
+    )
+    (property "Datasheet" "~" (at 195.58 123.19 0)
+      (effects (font (size 1.27 1.27)) hide)
+    )
+    (pin "1")
+    (pin "2")
+    (instances
+      (project "PDU"
+        (path "/e63e39d7-6ac0-4ffd-8aa3-1841a4541b55/e469982c-3823-4665-9e6d-e90b00c2da09"
+          (reference "C16") (unit 1)
+        )
+      )

Commit message: v2.2 hardware
Parts:
- removed R24: 10k, Resistor_SMD:R_0402_1005Metric, symbol Device:R_Small
- removed R26: 160k, Resistor_SMD:R_0402_1005Metric, symbol Device:R_Small
Connections:
- net LIPOPOWER: no longer names the net of U1.4 (STAT)
- net USBPOWER: no longer names the net of U8.4 (STAT)
- no-connect marks 3 -> 5
