File: Powerboard/Hardware/PDU.kicad_sch (KiCad schematic)
At the start: 46 parts, among them J1 Conn_01x03_MountingPin, J7 XT60PW-M, J8 Conn_01x04_Male, J9 XT60PW-M, U2 ESP32-S3, Y1 40MHz±10ppm

Commit message: shiven layout change
Parts:
- added C28: 0.1uF, Capacitor_SMD:C_0402_1005Metric, symbol Device:C_Small
- R14: value 47k -> 97.6k
Connections:
- net +12V: now also C28.1
- net ARMING: now also U2.41 (GPIO36); no longer U2.38 (GPIO33)
- net BattVoltage: now also U2.11 (GPIO6/ADC1_CH5), C28.2; no longer U2.19 (GPIO14/ADC2_CH3)
- net CAN_RX: now also U2.13 (GPIO8/ADC1_CH7); no longer U2.47 (MTDI/JTAG/GPIO41)
- net CAN_TX: now also U2.14 (GPIO9/ADC1_CH8); no longer U2.45 (MTDO/JTAG/GPIO40)
- net DepVoltage: now also U2.7 (GPIO2/ADC1_CH1); no longer U2.18 (GPIO13/ADC2_CH2)
- net LogicSwitch: now also U2.40 (GPIO35); no longer U2.41 (GPIO36)
- net LogicVoltage: now also U2.6 (GPIO1/ADC1_CH0); no longer U2.11 (GPIO6/ADC1_CH5)
- net SCL: now also U2.37 (SPICLK_P/GPIO47); no longer U2.44 (MTCK/JTAG/GPIO39)
- net SDA: now also U2.36 (SPICLK_N/GPIO48); no longer U2.43 (GPIO38)
- net DepCurrent: now reaches U2.10 (GPIO5/ADC1_CH4)
- net EFuse_PG: now reaches U2.9 (GPIO4/ADC1_CH3)
- no-connect marks 31 -> 29
Other:
- sheet Switches+RBUS ports: added DepCurrent, EFuse_PG; removed none
Changed lines of the file:
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@@
 	)
 	(junction
+		(at 61.468 142.494)
+		(diameter 0)
+		(color 0 0 0 0)
+	)
+	(junction
 		(at 273.812 132.842)
 		(diameter 0)
@@
 	)
 	(no_connect
+		(at 176.022 121.412)
+	)
+	(no_connect
 		(at 176.022 126.492)
 	)
@@
 	)
 	(no_connect
-		(at 242.062 116.332)
+		(at 242.062 108.712)
+	)
+	(no_connect
+		(at 176.022 123.952)
 	)
 	(no_connect
-		(at 242.062 118.872)
+		(at 176.022 118.872)
 	)
 	(no_connect
@@
 	)
 	(no_connect
-		(at 176.022 75.692)
-	)
-	(no_connect
-		(at 176.022 80.772)
+		(at 176.022 106.172)
 	)
 	(no_connect
-		(at 176.022 83.312)
-	)
-	(no_connect
-		(at 176.022 88.392)
-	)
-	(no_connect
-		(at 176.022 90.932)
-	)
-	(no_connect
-		(at 176.022 93.472)
+		(at 176.022 103.632)
 	)
 	(no_connect
@@
 	)
 	(no_connect
-		(at 242.062 101.092)
+		(at 242.062 96.012)
 	)
 	(no_connect
@@
 	)
 	(no_connect
-		(at 176.022 73.152)
+		(at 176.022 88.392)
 	)
 	(no_connect
@@
 	(wire
 		(pts
+			(xy 56.642 143.002) (xy 56.642 142.494)
+		)
+		(stroke
+			(width 0)
+			(type default)
+		)
+	)
+	(wire
+		(pts
 			(xy 176.022 127.762) (xy 176.022 131.572)
 		)
@@
 	(wire
 		(pts
+			(xy 56.642 142.494) (xy 61.468 142.494)
+		)
+		(stroke
+			(width 0)
+			(type default)
+		)
+	)
+	(wire
+		(pts
 			(xy 123.952 31.242) (xy 129.032 31.242)
 		)
@@
 	(wire
 		(pts
+			(xy 56.642 148.082) (xy 56.642 148.844)
+		)
+		(stroke
+			(width 0)
+			(type default)
+		)
+	)
+	(wire
+		(pts
 			(xy 122.682 170.942) (xy 122.682 172.212)
 		)
@@
 		)
 	)
+	(wire
+		(pts
+			(xy 56.642 148.844) (xy 61.468 148.844)
+		)
+		(stroke
+			(width 0)
+			(type default)
+		)
+	)
 	(polyline
 		(pts
@@
 	)
 	(label "BattVoltage"
-		(at 176.022 106.172 180)
+		(at 176.022 85.852 180)
 		(fields_autoplaced yes)
 		(effects
@@
 		)
 	)
+	(label "DepCurrent"
+		(at 176.022 83.312 180)
+		(fields_autoplaced yes)
+		(effects
+			(font
+				(size 1.27 1.27)
+			)
+			(justify right bottom)
+		)
+	)
+	(label "EFuse_PG"
+		(at 64.262 85.852 0)
+		(fields_autoplaced yes)
+		(effects
+			(font
+				(size 1.27 1.27)
+			)
+			(justify left bottom)
+		)
+	)
 	(label "CAN+"
 		(at 35.052 78.74 180)
@@
 	)
 	(label "SCL"
-		(at 176.022 118.872 180)
+		(at 242.062 118.872 0)
 		(fields_autoplaced yes)
 		(effects
@@
 				(size 1.27 1.27)
 			)
-			(justify right bottom)
+			(justify left bottom)
 		)
 	)
@@
 	)
 	(label "LogicSwitch"
-		(at 242.062 103.632 0)
+		(at 242.062 101.092 0)
+		(fields_autoplaced yes)
+		(effects
+			(font
+				(size 1.27 1.27)
+			)
+			(justify left bottom)
+		)
+	)
+	(label "DepCurrent"
+		(at 64.262 74.93 0)
 		(fields_autoplaced yes)
 		(effects
@@
 	)
 	(label "ARMING"
-		(at 242.062 96.012 0)
+		(at 242.062 103.632 0)
 		(fields_autoplaced yes)
 		(effects
@@
 		)
 	)
+	(label "EFuse_PG"
+		(at 176.022 80.772 180)
+		(fields_autoplaced yes)
+		(effects
+			(font
+				(size 1.27 1.27)
+			)
+			(justify right bottom)
+		)
+	)
 	(label "CHIP_PU"
 		(at 165.862 68.072 0)
@@
 	)
 	(label "SDA"
-		(at 242.062 108.712 0)
+		(at 242.062 116.332 0)
 		(fields_autoplaced yes)
 		(effects
@@
 	)
 	(label "LogicVoltage"
-		(at 176.022 85.852 180)
+		(at 176.022 73.152 180)
 		(fields_autoplaced yes)
 		(effects
@@
 	)
 	(label "CAN_TX"
-		(at 176.022 121.412 180)
+		(at 176.022 93.472 180)
 		(fields_autoplaced yes)
 		(effects
@@
 	)
 	(label "CAN_RX"
-		(at 176.022 123.952 180)
+		(at 176.022 90.932 180)
 		(fields_autoplaced yes)
 		(effects
@@
 	)
 	(label "DepVoltage"
-		(at 176.022 103.632 180)
+		(at 176.022 75.692 180)
 		(fields_autoplaced yes)
 		(effects
@@
 	(symbol
 		(lib_id "Device:C_Small")
+		(at 56.642 145.542 0)
+		(unit 1)
+		(exclude_from_sim no)
+		(in_bom yes)
+		(on_board yes)
+		(dnp no)
+		(property "Reference" "C28"
+			(at 49.276 144.6417 0)
+			(effects
+				(font
+					(size 1.27 1.27)
+				)
+				(justify left)
+			)
+		)
+		(property "Value" "0.1uF"
+			(at 49.276 147.066 0)
+			(effects
+				(font
+					(size 1.27 1.27)
+				)
+				(justify left)
+			)
+		)
+		(property "Footprint" "Capacitor_SMD:C_0402_1005Metric"
+			(at 56.642 145.542 0)
+			(effects
+				(font
+					(size 1.27 1.27)
+				)
+				(hide yes)
+			)
+		)
+		(property "Datasheet" "~"
+			(at 56.642 145.542 0)
+			(effects
+				(font
+					(size 1.27 1.27)
+				)
+				(hide yes)
+			)
+		)
+		(property "Description" "Unpolarized capacitor, small symbol"
+			(at 56.642 145.542 0)
+			(effects
+				(font
+					(size 1.27 1.27)
+				)
+				(hide yes)
+			)
+		)
+		(pin "2"
+		)
+		(pin "1"
+		)
+		(instances
+			(project "PDU"
+				(path "/e63e39d7-6ac0-4ffd-8aa3-1841a4541b55"
+					(reference "C28")
+					(unit 1)
+				)
+			)
+		)
+	)
+	(symbol
+		(lib_id "Device:C_Small")
 		(at 126.492 139.192 0)
 		(unit 1)
@@
 		(fields_autoplaced yes)
 		(property "Reference" "R14"
-			(at 62.9666 144.1993 0)
+			(at 62.9666 143.8218 0)
 			(effects
 				(font
@@
 			)
 		)
-		(property "Value" "47k"
-			(at 62.9666 146.7362 0)
+		(property "Value" "97.6k"
+			(at 62.9666 146.2461 0)
 			(effects
 				(font
@@
 			(effects
 				(font
+					(size 1.27 1.27)
+				)
+				(justify right)
+			)
+		)
+		(pin "DepCurrent" output
+			(at 64.262 74.93 0)
+			(effects
+				(font
+					(size 1.27 1.27)
+				)
+				(justify right)
+			)
+		)
+		(pin "EFuse_PG" output
+			(at 64.262 85.852 0)
+			(effects
+				(font

Commit message: changes post 3rd review
Parts:
- J1: footprint iclr:Molex_Nano-Fit_105313-xx02_1x02_P2.50mm_Horizontal -> Connector_Molex:Molex_Nano-Fit_105313-xx02_1x02_P2.50mm_Horizontal
Changed lines of the file:
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@@
 			)
 		)
-		(property "Footprint" "iclr:Molex_Nano-Fit_105313-xx02_1x02_P2.50mm_Horizontal"
+		(property "Footprint" "Connector_Molex:Molex_Nano-Fit_105313-xx02_1x02_P2.50mm_Horizontal"
 			(at 32.258 134.874 0)
 			(effects
@@
 			)
 		)
-		(property "Description" ""
+		(property "Description" "Generic connectable mounting pin connector, single row, 01x03, script generated (kicad-library-utils/schlib/autogen/connector/)"
 			(at 32.258 134.874 0)
 			(effects
