File: Powerboard/Hardware/3v3filter.kicad_sch (KiCad schematic)
At the start: 17 parts, among them U10 SC4215, U4 MAX77827AEFD+T

Commit message: new layout
Connections:
- net GNDA is gone; now on net GND: C49.2, R1.2, U4.4 (AGND)
Changed lines of the file:
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@@
   (junction (at 155.702 69.85) (diameter 0) (color 0 0 0 0)
+  )
+  (junction (at 153.162 92.71) (diameter 0) (color 0 0 0 0)
   )
   (junction (at 170.942 69.85) (diameter 0) (color 0 0 0 0)
@@
   )
   (wire (pts (xy 187.452 69.85) (xy 187.452 78.74))
+    (stroke (width 0) (type default))
+  )
+  (wire (pts (xy 153.162 92.71) (xy 155.956 92.71))
     (stroke (width 0) (type default))
   )
@@
     (effects (font (size 1.27 1.27)) (justify left bottom))
   )
+  (label "GNDA" (at 155.956 92.71 0) (fields_autoplaced)
+    (effects (font (size 1.27 1.27)) (justify left bottom))
+  )

Commit message: v2.1 ordering
Parts:
- R12: value 470 -> 5.1k
- USBLED1: value USB_LED -> WHITE_LED
Changed lines of the file:
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@@
       (effects (font (size 1.27 1.27)))
     )
-    (property "Value" "USB_LED" (at 145.034 102.2604 0)
+    (property "Value" "WHITE_LED" (at 145.034 102.2604 0)
       (effects (font (size 1.27 1.27)))
     )
@@
       (effects (font (size 1.27 1.27)))
     )
-    (property "Value" "470" (at 137.414 107.823 90)
-      (effects (font (size 1.27 1.27)))
-    )
+    (property "Value" "5.1k" (at 137.414 107.823 90)
+      (effects (font (size 1.27 1.27)))
+    )

Commit message: v2.2 hardware
Parts:
- removed TP3, TP6: TestPoint, TestPoint:TestPoint_Pad_D1.0mm, symbol Connector:TestPoint
