File: Powerboard/Hardware/usb.kicad_sch (KiCad schematic)
At the start: 6 parts, among them J3 USB_C_Receptacle_USB2.0

Commit message: v2.2 hardware
Parts:
- removed TP1, TP2: TestPoint, TestPoint:TestPoint_Pad_D1.0mm, symbol Connector:TestPoint
