File: Hardware/PDU.kicad_sch (KiCad schematic)
At the start: 47 parts, among them J1 Conn_01x03_MountingPin, J7 XT60PW-M, J8 Conn_01x04_Male, J9 XT60PW-M, U2 ESP32-S3, Y1 40MHz±10ppm

Commit message: Initial changes : removed efuse in place of a current sensor and hardware fuse xt60
Parts:
- renumbered C28 to C1, C9 to C10, C10 to C11, C11 to C12, C1 to C2, C2 to C3, C3 to C4, C4 to C5, C5 to C6, C6 to C7, C7 to C8, C8 to C9, J8 to J2, J9 to J3, J7 to J4, R14 to R1, R9 to R10, R46 to R11, R8 to R12, R22 to R2, R26 to R3, R27 to R4, R3 to R5, R5 to R6, R6 to R7, R7 to R8, R4 to R9, TP5 to TP1, TP4 to TP2, U2 to U1
Connections:
- net CUR_SENS_SCL: now reaches U1.15 (GPIO10/ADC1_CH9)
- net CUR_SENS_SDA: now reaches U1.16 (GPIO11/ADC2_CH0)
- net DepCurrent: no longer names the net of U1.10 (GPIO5/ADC1_CH4)
- net EFuse_PG: no longer names the net of U1.9 (GPIO4/ADC1_CH3)
Other:
- sheet Switches+RBUS ports: added CUR_SENS_SCL, CUR_SENS_SDA; removed DepCurrent, EFuse_PG

Commit message: cleaned up schematic and bom
Parts:
- C101: renamed from C1; value 0.1uF -> 100nF
- C104: renamed from C4; value 0.1uF -> 100nF
- C106: renamed from C6; value 0.1uF -> 100nF
- C107: renamed from C7; value 0.1uF -> 100nF
- C109: renamed from C9; value 0.1uF -> 100nF
- C111: renamed from C11; value 0.1uF -> 100nF
- C112: renamed from C12; value 0.1uF -> 100nF
- D101: renamed from CANTXLED1; value EMERALD_LED -> LED_GREEN
- D102: renamed from CANRXLED1; value ORANGE_LED -> LED_ORANGE
- D103: renamed from TXLED1; value GREEN_LED -> LED_GREEN
- D104: renamed from 3V3LED1; value CYAN_LED -> LED_BLUE
- D105: renamed from BATTLED1; value ORANGE_LED -> LED_ORANGE
- H101: renamed from H1; now left out of the parts list
- H102: renamed from H2; now left out of the parts list
- H103: renamed from H3; now left out of the parts list
- H104: renamed from H4; now left out of the parts list
- L101: renamed from L1; value 2.0nH -> 2nH
- R101: renamed from R1; value 97.6k -> 97.6kΩ
- R102: renamed from R2; value 10k -> 10kΩ
- R103: renamed from R3; value 1k -> 1kΩ
- R104: renamed from R4; value 1k -> 1kΩ
- R105: renamed from R5; value 10K -> 10kΩ
- R106: renamed from R6; value 470 -> 470Ω
- R107: renamed from R7; value 10K -> 10kΩ
- R108: renamed from R8; value 470 -> 470Ω
- R109: renamed from R9; value 499 -> 499Ω
- R110: renamed from R10; value 3k -> 3kΩ
- R111: renamed from R11; value 2.2k -> 2.2kΩ
- R112: renamed from R12; value 2.2k -> 2.2kΩ
- TP101: renamed from TP1; now left out of the parts list
- TP102: renamed from TP2; now left out of the parts list
- renumbered C2 to C102, C3 to C103, C5 to C105, C8 to C108, C10 to C110, C13 to C113, C14 to C114, J1 to J101, J2 to J102, ENJUMPER1 to J103, BOOTJUMPER1 to J104, J3 to J105, J4 to J106, L2 to L102, U1 to U101, Y1 to Y101
