File: Hardware/can.kicad_sch (KiCad schematic)
At the start: 9 parts, among them U5 SN65HVD230

Commit message: Initial changes : removed efuse in place of a current sensor and hardware fuse xt60
Parts:
- renumbered C18 to C22, C19 to C23, C20 to C24, D2 to D1, R15 to R17, R23 to R18, R16 to R19, R17 to R20, U5 to U4
Changed lines of the file:
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@@
 (kicad_sch
-	(version 20231120)
+	(version 20250114)
 	(generator "eeschema")
-	(generator_version "8.0")
+	(generator_version "9.0")
 	(paper "A4")
 	(junction
@@
 	(label "Vref"
 		(at 137.16 92.456 180)
-		(fields_autoplaced yes)
 		(effects
 			(font
@@
 	(label "Vref"
 		(at 107.95 93.726 180)
-		(fields_autoplaced yes)
 		(effects
 			(font
@@
 		(shape output)
 		(at 95.25 88.646 180)
-		(fields_autoplaced yes)
 		(effects
 			(font
@@
 		(shape bidirectional)
 		(at 158.75 83.566 0)
-		(fields_autoplaced yes)
 		(effects
 			(font
@@
 		(shape bidirectional)
 		(at 173.99 83.566 0)
-		(fields_autoplaced yes)
 		(effects
 			(font
@@
 		(shape bidirectional)
 		(at 158.75 101.346 0)
-		(fields_autoplaced yes)
 		(effects
 			(font
@@
 		(shape input)
 		(at 95.25 91.186 180)
-		(fields_autoplaced yes)
 		(effects
 			(font
@@
 		(shape bidirectional)
 		(at 173.99 101.346 0)
-		(fields_autoplaced yes)
 		(effects
 			(font
@@
 		(dnp no)
 		(fields_autoplaced yes)
-		(property "Reference" "D2"
+		(property "Reference" "D1"
 			(at 173.99 91.186 90)
 			(effects
@@
 			(project "PDU"
 				(path "/e63e39d7-6ac0-4ffd-8aa3-1841a4541b55/12646a0c-a158-4f1c-9172-cd278d717c5e"
-					(reference "D2")
+					(reference "D1")
 					(unit 1)
 				)
@@
 		(on_board yes)
 		(dnp no)
-		(property "Reference" "R15"
+		(property "Reference" "R17"
 			(at 101.6 97.536 0)
 			(effects
@@
 			(project "PDU"
 				(path "/e63e39d7-6ac0-4ffd-8aa3-1841a4541b55/12646a0c-a158-4f1c-9172-cd278d717c5e"
-					(reference "R15")
+					(reference "R17")
 					(unit 1)
 				)
@@
 		(dnp no)
 		(fields_autoplaced yes)
-		(property "Reference" "C18"
+		(property "Reference" "C22"
 			(at 97.79 73.406 0)
 			(effects
@@
 			(project "PDU"
 				(path "/e63e39d7-6ac0-4ffd-8aa3-1841a4541b55/12646a0c-a158-4f1c-9172-cd278d717c5e"
-					(reference "C18")
+					(reference "C22")
 					(unit 1)
 				)
@@
 		(dnp no)
 		(fields_autoplaced yes)
-		(property "Reference" "#PWR0137"
+		(property "Reference" "#PWR038"
 			(at 107.95 75.946 0)
 			(effects
@@
 			(project "PDU"
 				(path "/e63e39d7-6ac0-4ffd-8aa3-1841a4541b55/12646a0c-a158-4f1c-9172-cd278d717c5e"
-					(reference "#PWR0137")
+					(reference "#PWR038")
 					(unit 1)
 				)
@@
 		(dnp no)
 		(fields_autoplaced yes)
-		(property "Reference" "R17"
+		(property "Reference" "R20"
 			(at 146.05 96.266 0)
 			(effects
@@
 			(project "PDU"
 				(path "/e63e39d7-6ac0-4ffd-8aa3-1841a4541b55/12646a0c-a158-4f1c-9172-cd278d717c5e"
-					(reference "R17")
+					(reference "R20")
 					(unit 1)
 				)
@@
 		(dnp no)
 		(fields_autoplaced yes)
-		(property "Reference" "#PWR0138"
+		(property "Reference" "#PWR039"
 			(at 107.95 83.566 0)
 			(effects
@@
 			(project "PDU"
 				(path "/e63e39d7-6ac0-4ffd-8aa3-1841a4541b55/12646a0c-a158-4f1c-9172-cd278d717c5e"
-					(reference "#PWR0138")
+					(reference "#PWR039")
 					(unit 1)
 				)
@@
 		(dnp no)
 		(fields_autoplaced yes)
-		(property "Reference" "#PWR0136"
+		(property "Reference" "#PWR040"
 			(at 118.11 108.966 0)
 			(effects
@@
 			(project "PDU"
 				(path "/e63e39d7-6ac0-4ffd-8aa3-1841a4541b55/12646a0c-a158-4f1c-9172-cd278d717c5e"
-					(reference "#PWR0136")
+					(reference "#PWR040")
 					(unit 1)
 				)
@@
 		(dnp no)
 		(fields_autoplaced yes)
-		(property "Reference" "C19"
+		(property "Reference" "C23"
 			(at 113.03 73.4122 0)
 			(effects
@@
 			(project "PDU"
 				(path "/e63e39d7-6ac0-4ffd-8aa3-1841a4541b55/12646a0c-a158-4f1c-9172-cd278d717c5e"
-					(reference "C19")
+					(reference "C23")
 					(unit 1)
 				)
@@
 		(dnp no)
 		(fields_autoplaced yes)
-		(property "Reference" "R16"
+		(property "Reference" "R19"
 			(at 146.05 86.106 0)
 			(effects
@@
 			(project "PDU"
 				(path "/e63e39d7-6ac0-4ffd-8aa3-1841a4541b55/12646a0c-a158-4f1c-9172-cd278d717c5e"
-					(reference "R16")
+					(reference "R19")
 					(unit 1)
 				)
@@
 		(dnp no)
 		(fields_autoplaced yes)
-		(property "Reference" "C20"
+		(property "Reference" "C24"
 			(at 154.94 86.106 90)
 			(effects
@@
 			(project "PDU"
 				(path "/e63e39d7-6ac0-4ffd-8aa3-1841a4541b55/12646a0c-a158-4f1c-9172-cd278d717c5e"
-					(reference "C20")
+					(reference "C24")
 					(unit 1)
 				)
@@
 		(dnp no)
 		(fields_autoplaced yes)
-		(property "Reference" "U5"
+		(property "Reference" "U4"
 			(at 125.73 78.7146 0)
 			(effects
@@
 			(project "PDU"
 				(path "/e63e39d7-6ac0-4ffd-8aa3-1841a4541b55/12646a0c-a158-4f1c-9172-cd278d717c5e"
-					(reference "U5")
+					(reference "U4")
 					(unit 1)
 				)
@@
 		(dnp no)
 		(fields_autoplaced yes)
-		(property "Reference" "R23"
+		(property "Reference" "R18"
 			(at 140.97 87.7402 90)
 			(effects
@@
 			(project "PDU"
 				(path "/e63e39d7-6ac0-4ffd-8aa3-1841a4541b55/12646a0c-a158-4f1c-9172-cd278d717c5e"
-					(reference "R23")
+					(reference "R18")
 					(unit 1)
 				)
@@
 		(dnp no)
 		(fields_autoplaced yes)
-		(property "Reference" "#PWR0140"
+		(property "Reference" "#PWR041"
 			(at 158.75 98.806 0)
 			(effects
@@
 			(project "PDU"
 				(path "/e63e39d7-6ac0-4ffd-8aa3-1841a4541b55/12646a0c-a158-4f1c-9172-cd278d717c5e"
-					(reference "#PWR0140")
-					(unit 1)
-				)
+					(reference "#PWR041")
+					(unit 1)
+				)

Commit message: cleaned up schematic and bom
Parts:
- R405: renamed from R17; value 0 -> 0Ω
- R409: renamed from R18; value 0 -> 0Ω
- R410: renamed from R19; value 60 -> 60Ω
- R411: renamed from R20; value 60 -> 60Ω
- renumbered C22 to C403, C23 to C404, C24 to C406, D1 to D403, U4 to U402
Changed lines of the file:
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@@
 		(dnp no)
 		(fields_autoplaced yes)
-		(property "Reference" "D1"
+		(property "Reference" "D403"
 			(at 173.99 91.186 90)
 			(effects
@@
 			(project "PDU"
 				(path "/e63e39d7-6ac0-4ffd-8aa3-1841a4541b55/12646a0c-a158-4f1c-9172-cd278d717c5e"
-					(reference "D1")
+					(reference "D403")
 					(unit 1)
 				)
@@
 		(on_board yes)
 		(dnp no)
-		(property "Reference" "R17"
+		(property "Reference" "R405"
 			(at 101.6 97.536 0)
 			(effects
@@
 			)
 		)
-		(property "Value" "0"
+		(property "Value" "0Ω"
 			(at 101.6 100.076 0)
 			(effects
@@
 			(project "PDU"
 				(path "/e63e39d7-6ac0-4ffd-8aa3-1841a4541b55/12646a0c-a158-4f1c-9172-cd278d717c5e"
-					(reference "R17")
+					(reference "R405")
 					(unit 1)
 				)
@@
 		(dnp no)
 		(fields_autoplaced yes)
-		(property "Reference" "C22"
+		(property "Reference" "C403"
 			(at 97.79 73.406 0)
 			(effects
@@
 			(project "PDU"
 				(path "/e63e39d7-6ac0-4ffd-8aa3-1841a4541b55/12646a0c-a158-4f1c-9172-cd278d717c5e"
-					(reference "C22")
+					(reference "C403")
 					(unit 1)
 				)
@@
 		(dnp no)
 		(fields_autoplaced yes)
-		(property "Reference" "#PWR038"
+		(property "Reference" "#PWR0408"
 			(at 107.95 75.946 0)
 			(effects
@@
 			(project "PDU"
 				(path "/e63e39d7-6ac0-4ffd-8aa3-1841a4541b55/12646a0c-a158-4f1c-9172-cd278d717c5e"
-					(reference "#PWR038")
+					(reference "#PWR0408")
 					(unit 1)
 				)
@@
 		(dnp no)
 		(fields_autoplaced yes)
-		(property "Reference" "R20"
+		(property "Reference" "R411"
 			(at 146.05 96.266 0)
 			(effects
@@
 			)
 		)
-		(property "Value" "60"
+		(property "Value" "60Ω"
 			(at 146.05 98.806 0)
 			(effects
@@
 			(project "PDU"
 				(path "/e63e39d7-6ac0-4ffd-8aa3-1841a4541b55/12646a0c-a158-4f1c-9172-cd278d717c5e"
-					(reference "R20")
+					(reference "R411")
 					(unit 1)
 				)
@@
 		(dnp no)
 		(fields_autoplaced yes)
-		(property "Reference" "#PWR039"
+		(property "Reference" "#PWR0409"
 			(at 107.95 83.566 0)
 			(effects
@@
 			(project "PDU"
 				(path "/e63e39d7-6ac0-4ffd-8aa3-1841a4541b55/12646a0c-a158-4f1c-9172-cd278d717c5e"
-					(reference "#PWR039")
+					(reference "#PWR0409")
 					(unit 1)
 				)
@@
 		(dnp no)
 		(fields_autoplaced yes)
-		(property "Reference" "#PWR040"
+		(property "Reference" "#PWR0413"
 			(at 118.11 108.966 0)
 			(effects
@@
 			(project "PDU"
 				(path "/e63e39d7-6ac0-4ffd-8aa3-1841a4541b55/12646a0c-a158-4f1c-9172-cd278d717c5e"
-					(reference "#PWR040")
+					(reference "#PWR0413")
 					(unit 1)
 				)
@@
 		(dnp no)
 		(fields_autoplaced yes)
-		(property "Reference" "C23"
+		(property "Reference" "C404"
 			(at 113.03 73.4122 0)
 			(effects
@@
 			(project "PDU"
 				(path "/e63e39d7-6ac0-4ffd-8aa3-1841a4541b55/12646a0c-a158-4f1c-9172-cd278d717c5e"
-					(reference "C23")
+					(reference "C404")
 					(unit 1)
 				)
@@
 		(dnp no)
 		(fields_autoplaced yes)
-		(property "Reference" "R19"
+		(property "Reference" "R410"
 			(at 146.05 86.106 0)
 			(effects
@@
 			)
 		)
-		(property "Value" "60"
+		(property "Value" "60Ω"
 			(at 146.05 88.646 0)
 			(effects
@@
 			(project "PDU"
 				(path "/e63e39d7-6ac0-4ffd-8aa3-1841a4541b55/12646a0c-a158-4f1c-9172-cd278d717c5e"
-					(reference "R19")
+					(reference "R410")
 					(unit 1)
 				)
@@
 		(dnp no)
 		(fields_autoplaced yes)
-		(property "Reference" "C24"
+		(property "Reference" "C406"
 			(at 154.94 86.106 90)
 			(effects
@@
 			(project "PDU"
 				(path "/e63e39d7-6ac0-4ffd-8aa3-1841a4541b55/12646a0c-a158-4f1c-9172-cd278d717c5e"
-					(reference "C24")
+					(reference "C406")
 					(unit 1)
 				)
@@
 		(dnp no)
 		(fields_autoplaced yes)
-		(property "Reference" "U4"
+		(property "Reference" "U402"
 			(at 125.73 78.7146 0)
 			(effects
@@
 			(project "PDU"
 				(path "/e63e39d7-6ac0-4ffd-8aa3-1841a4541b55/12646a0c-a158-4f1c-9172-cd278d717c5e"
-					(reference "U4")
+					(reference "U402")
 					(unit 1)
 				)
@@
 		(dnp no)
 		(fields_autoplaced yes)
-		(property "Reference" "R18"
+		(property "Reference" "R409"
 			(at 140.97 87.7402 90)
 			(effects
@@
 			)
 		)
-		(property "Value" "0"
+		(property "Value" "0Ω"
 			(at 140.97 90.2771 90)
 			(effects
@@
 			(project "PDU"
 				(path "/e63e39d7-6ac0-4ffd-8aa3-1841a4541b55/12646a0c-a158-4f1c-9172-cd278d717c5e"
-					(reference "R18")
+					(reference "R409")
 					(unit 1)
 				)
@@
 		(dnp no)
 		(fields_autoplaced yes)
-		(property "Reference" "#PWR041"
+		(property "Reference" "#PWR0416"
 			(at 158.75 98.806 0)
 			(effects
@@
 			(project "PDU"
 				(path "/e63e39d7-6ac0-4ffd-8aa3-1841a4541b55/12646a0c-a158-4f1c-9172-cd278d717c5e"
-					(reference "#PWR041")
-					(unit 1)
-				)
+					(reference "#PWR0416")
+					(unit 1)
+				)
