File: Hardware/switches.kicad_sch (KiCad schematic)
At the start: 38 parts, among them IC1 TPS259830ONRGER, J2 FAN, J4 Conn_01x02_Male, J5 Conn_01x08_Male, J6 Conn_01x02_Male, Q1 SSM3K15AMFV,L3F, Q2 SI7635DP-T1-GE3, Q3 SI7635DP-T1-GE3, Q7 SQS141ELNW-T1_GE3, Q8 SQS141ELNW-T1_GE3, U6 LTC4412xS6, U7 LTC4412xS6

Commit message: Initial changes : removed efuse in place of a current sensor and hardware fuse xt60
Parts:
- removed C21: 4.7nF, Capacitor_SMD:C_0402_1005Metric, symbol Device:C_Small
- removed C22: 10nF, Capacitor_SMD:C_0402_1005Metric, symbol Device:C_Small
- removed D4: SMCJ24AHE3_A/H, Diode_SMD:D_SMC, symbol Diode:PTVS5V0Z1USK
- removed IC1: TPS259830ONRGER, iclr:TPS259830ONRGER, symbol iclr:TPS259830ONRGER
- removed R38: 82, Capacitor_SMD:C_0402_1005Metric, symbol Device:R_Small
- removed R39: 1M, Capacitor_SMD:C_0402_1005Metric, symbol Device:R_Small
- removed R40: 732k, Capacitor_SMD:C_0402_1005Metric, symbol Device:R_Small
- removed R41: 73.2k, Capacitor_SMD:C_0402_1005Metric, symbol Device:R_Small
- removed R42: 680, Capacitor_SMD:C_0402_1005Metric, symbol Device:R_Small
- removed R43: 100k, Capacitor_SMD:C_0402_1005Metric, symbol Device:R_Small
- added C29, C30: 0.1uF, Capacitor_SMD:C_0402_1005Metric, symbol Device:C_Small
- added J8: XT60PW-F, AMASS_XT60PW-F, symbol iclr:XT60PW-F
- added R28: 2m, Resistor_SMD:R_2512_6332Metric_Pad1.40x3.35mm_HandSolder, symbol Device:R
- added R29: 10k, Resistor_SMD:R_0402_1005Metric, symbol Device:R_Small
- added R30, R31: 10, Resistor_SMD:R_0402_1005Metric, symbol Device:R_Small
- added R34, R35: 3.3k, Resistor_SMD:R_0402_1005Metric, symbol Device:R_Small
- added TP3, TP4: TestPoint, TestPoint:TestPoint_Pad_D1.0mm, symbol Connector:TestPoint
- added U7: INA219AxDCN, Package_TO_SOT_SMD:SOT-23-8, symbol Sensor_Energy:INA219AxDCN
- renumbered C23 to C25, C24 to C28, J4 to J5, J5 to J6, J2 to J7, J6 to J9, JP2 to JP1, JP1 to JP2, Q7 to Q1, Q8 to Q2, Q2 to Q3, Q3 to Q4, Q1 to Q5, R18 to R21, R24 to R22, R26 to R23, R33 to R24, R27 to R25, R28 to R26, R32 to R27, R39 to R32, R38 to R33, U6 to U5, U7 to U6
Connections:
- net +12V: now also J8.2
- net +3V3: now also C30.1, R34.1, R35.1, U7.4 (VS)
- net GND: now also C30.2, J8.S1 (SHIELD), J8.S2 (SHIELD), R29.1, U7.3 (GND), U7.7 (A0), U7.8 (A1)
- net EFuse_OUT renamed Fuse_OUT
- net Fuse_OUT: now also R28.2, R29.2, R31.1
- new net: J8.1, R28.1, R30.1
- new net CUR_SENS_SCL: R35.2, TP4.1, U7.5 (SCL)
- new net CUR_SENS_SDA: R34.2, TP3.1, U7.6 (SDA)
- new net SHNT_IN+: C29.1, R30.2, U7.1 (IN+)
- new net SHNT_IN-: C29.2, R31.2, U7.2 (IN-)
- no-connect marks 4 -> 2
Other:
- note added: "XT-60 To Fuse"
- note removed: "UV set to 2.7V OV set to 30V"
- note removed: "dvdt pin left floating for fastest turn on time"

Commit message: cleaned up schematic and bom
Parts:
- C401: renamed from C25; value 1000uF -> 1mF
- C402: renamed from C26; value 0.1uF -> 100nF
- C405: renamed from C27; value 0.1uF -> 100nF
- C408: renamed from C29; value 0.1uF -> 100nF
- C409: renamed from C30; value 0.1uF -> 100nF
- D401: renamed from LOGICLED1; value BLUE_LED -> LED_BLUE
- D402: renamed from DEPLED1; value RED_LED -> LED_RED
- JP401: renamed from JP1; now left out of the parts list
- JP402: renamed from JP2; now left out of the parts list
- R401: renamed from R21; value 10k -> 10kΩ
- R402: renamed from R22; value 2.87k -> 2.87kΩ
- R403: renamed from R23; value 10k -> 10kΩ
- R404: renamed from R24; value 470 -> 470Ω
- R406: renamed from R25; value 3k -> 3kΩ
- R407: renamed from R26; value 97.6k -> 97.6kΩ
- R408: renamed from R27; value 10k -> 10kΩ
- R412: renamed from R28; value 2m -> 2mΩ
- R413: renamed from R29; value 10k -> 10kΩ
- R414: renamed from R30; value 10 -> 10Ω
- R415: renamed from R31; value 10 -> 10Ω
- R416: renamed from R32; value 1k -> 1kΩ
- R417: renamed from R33; value 10k -> 10kΩ
- R418: renamed from R34; value 3.3k -> 3.3kΩ
- R419: renamed from R35; value 3.3k -> 3.3kΩ
- TP401: renamed from TP3; now left out of the parts list
- TP402: renamed from TP4; now left out of the parts list
- renumbered C28 to C407, J5 to J401, J6 to J402, J7 to J403, J8 to J404, J9 to J405, Q1 to Q401, Q2 to Q402, Q3 to Q403, Q4 to Q404, Q5 to Q405, U5 to U401, U6 to U403, U7 to U404
