File: Hardware/3v3bucks.kicad_sch (KiCad schematic)
At the start: 28 parts, among them IC2 SiC437AED-T1-GE3, Q5 PXP012-30QLJ, Q6 PXP012-30QLJ, U1 LTC4412xS6, U8 LTC4412xS6

Commit message: Initial changes : removed efuse in place of a current sensor and hardware fuse xt60
Parts:
- renumbered C15 to C31, C25 to C32, C30 to C33, C32 to C34, C34 to C35, C38 to C37, C47 to C38, C40 to C39, C42 to C40, C44 to C41, C46 to C42, C16 to C43, C12 to C44, IC2 to IC1, L3 to L4, Q5 to Q6, Q6 to Q7, R20 to R38, R21 to R39, R25 to R40, R29 to R41, R30 to R42, R31 to R43, R37 to R44, R47 to R45, U1 to U8, U8 to U9

Commit message: cleaned up schematic and bom
Parts:
- C210: renamed from C40; value 0.1uF -> 100nF
- L201: renamed from L4; value SRP1050WA-3R3M -> 3.3uH
- R201: renamed from R38; value 45.3k -> 45.3kΩ
- R202: renamed from R39; value 10k -> 10kΩ
- R203: renamed from R40; value 10k -> 10kΩ
- R204: renamed from R41; value 51k -> 51kΩ
- R205: renamed from R42; value 2.2 -> 2.2Ω
- R206: renamed from R43; value 100k -> 100kΩ
- R208: renamed from R45; value 100k -> 100kΩ
- renumbered C31 to C201, C32 to C202, C33 to C203, C34 to C204, C35 to C205, C36 to C206, C37 to C207, C38 to C208, C39 to C209, C41 to C211, C42 to C212, C43 to C213, C44 to C214, Q6 to Q201, Q7 to Q202, R44 to R207, IC1 to U201, U8 to U202, U9 to U203

Commit message: continued
Parts:
- U201: value SiC437AED-T1-GE3 -> SIC437AED-T1-GE3
Changed lines of the file:
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@@
 			)
 		)
-		(property "Value" "SiC437AED-T1-GE3"
+		(property "Value" "SIC437AED-T1-GE3"
 			(at 133.096 87.63 0)
 			(effects
