File: Hardware/3v3filter.kicad_sch (KiCad schematic)
At the start: 15 parts, among them U10 SC4215, U4 MAX77827AEFD+T

Commit message: Initial changes : removed efuse in place of a current sensor and hardware fuse xt60
Parts:
- renumbered C17 to C15, C49 to C16, C50 to C17, C51 to C18, C52 to C19, C53 to C20, C54 to C21, L5 to L3, R1 to R13, R12 to R14, R2 to R15, R13 to R16, U4 to U2, U10 to U3
Changed lines of the file:
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@@
 (kicad_sch
-	(version 20231120)
+	(version 20250114)
 	(generator "eeschema")
-	(generator_version "8.0")
+	(generator_version "9.0")
 	(paper "A4")
 	(junction
@@
 	(label "GNDA"
 		(at 158.242 90.17 0)
-		(fields_autoplaced yes)
 		(effects
 			(font
@@
 	(label "BIAS"
 		(at 118.872 85.09 180)
-		(fields_autoplaced yes)
 		(effects
 			(font
@@
 	(label "BBOUT"
 		(at 156.972 69.85 0)
-		(fields_autoplaced yes)
 		(effects
 			(font
@@
 	(label "SEL"
 		(at 112.522 82.55 180)
-		(fields_autoplaced yes)
 		(effects
 			(font
@@
 	(label "GNDA"
 		(at 112.522 87.63 270)
-		(fields_autoplaced yes)
 		(effects
 			(font
@@
 	(label "FBIn"
 		(at 223.012 78.74 180)
-		(fields_autoplaced yes)
 		(effects
 			(font
@@
 	(label "GNDA"
 		(at 118.872 90.17 270)
-		(fields_autoplaced yes)
 		(effects
 			(font
@@
 	(label "LX2"
 		(at 153.162 82.55 0)
-		(fields_autoplaced yes)
 		(effects
 			(font
@@
 	(label "BBIN"
 		(at 118.872 69.85 180)
-		(fields_autoplaced yes)
 		(effects
 			(font
@@
 	(label "LX1"
 		(at 153.162 74.93 0)
-		(fields_autoplaced yes)
 		(effects
 			(font
@@
 	(label "GNDA"
 		(at 155.956 92.71 0)
-		(fields_autoplaced yes)
 		(effects
 			(font
@@
 		(on_board yes)
 		(dnp no)
-		(property "Reference" "#PWR0128"
+		(property "Reference" "#PWR031"
 			(at 153.924 105.156 0)
 			(effects
@@
 			(project "PDU"
 				(path "/e63e39d7-6ac0-4ffd-8aa3-1841a4541b55/12e3318b-d723-448e-80f4-0a2add1fb722"
-					(reference "#PWR0128")
+					(reference "#PWR031")
 					(unit 1)
 				)
@@
 		(on_board yes)
 		(dnp no)
-		(property "Reference" "#PWR0189"
+		(property "Reference" "#PWR037"
 			(at 242.062 81.28 0)
 			(effects
@@
 			(project "PDU"
 				(path "/e63e39d7-6ac0-4ffd-8aa3-1841a4541b55/12e3318b-d723-448e-80f4-0a2add1fb722"
-					(reference "#PWR0189")
+					(reference "#PWR037")
 					(unit 1)
 				)
@@
 		(dnp no)
 		(fields_autoplaced yes)
-		(property "Reference" "#PWR0146"
+		(property "Reference" "#PWR029"
 			(at 115.062 81.28 0)
 			(effects
@@
 			(project "PDU"
 				(path "/e63e39d7-6ac0-4ffd-8aa3-1841a4541b55/12e3318b-d723-448e-80f4-0a2add1fb722"
-					(reference "#PWR0146")
+					(reference "#PWR029")
 					(unit 1)
 				)
@@
 		(on_board yes)
 		(dnp no)
-		(property "Reference" "C51"
+		(property "Reference" "C18"
 			(at 173.2661 71.5616 0)
 			(effects
@@
 			(project "PDU"
 				(path "/e63e39d7-6ac0-4ffd-8aa3-1841a4541b55/12e3318b-d723-448e-80f4-0a2add1fb722"
-					(reference "C51")
+					(reference "C18")
 					(unit 1)
 				)
@@
 		(on_board yes)
 		(dnp no)
-		(property "Reference" "C53"
+		(property "Reference" "C20"
 			(at 233.172 72.39 0)
 			(effects
@@
 			(project "PDU"
 				(path "/e63e39d7-6ac0-4ffd-8aa3-1841a4541b55/12e3318b-d723-448e-80f4-0a2add1fb722"
-					(reference "C53")
+					(reference "C20")
 					(unit 1)
 				)
@@
 		(on_board yes)
 		(dnp no)
-		(property "Reference" "C17"
+		(property "Reference" "C15"
 			(at 107.442 72.39 0)
 			(effects
@@
 			(project "PDU"
 				(path "/e63e39d7-6ac0-4ffd-8aa3-1841a4541b55/12e3318b-d723-448e-80f4-0a2add1fb722"
-					(reference "C17")
+					(reference "C15")
 					(unit 1)
 				)
@@
 		(dnp no)
 		(fields_autoplaced yes)
-		(property "Reference" "U10"
+		(property "Reference" "U3"
 			(at 205.232 63.7372 0)
 			(effects
@@
 			(project "PDU"
 				(path "/e63e39d7-6ac0-4ffd-8aa3-1841a4541b55/12e3318b-d723-448e-80f4-0a2add1fb722"
-					(reference "U10")
+					(reference "U3")
 					(unit 1)
 				)
@@
 		(on_board yes)
 		(dnp no)
-		(property "Reference" "R1"
+		(property "Reference" "R13"
 			(at 107.442 83.82 0)
 			(effects
@@
 			(project "PDU"
 				(path "/e63e39d7-6ac0-4ffd-8aa3-1841a4541b55/12e3318b-d723-448e-80f4-0a2add1fb722"
-					(reference "R1")
+					(reference "R13")
 					(unit 1)
 				)
@@
 		(on_board yes)
 		(dnp no)
-		(property "Reference" "C54"
+		(property "Reference" "C21"
 			(at 247.5603 71.6954 0)
 			(effects
@@
 			(project "PDU"
 				(path "/e63e39d7-6ac0-4ffd-8aa3-1841a4541b55/12e3318b-d723-448e-80f4-0a2add1fb722"
-					(reference "C54")
+					(reference "C21")
 					(unit 1)
 				)
@@
 		(dnp no)
 		(fields_autoplaced yes)
-		(property "Reference" "U4"
+		(property "Reference" "U2"
 			(at 137.922 63.6102 0)
 			(effects
@@
 			(project "PDU"
 				(path "/e63e39d7-6ac0-4ffd-8aa3-1841a4541b55/12e3318b-d723-448e-80f4-0a2add1fb722"
-					(reference "U4")
+					(reference "U2")
 					(unit 1)
 				)
@@
 		(dnp no)
 		(fields_autoplaced yes)
-		(property "Reference" "#PWR0187"
+		(property "Reference" "#PWR035"
 			(at 226.822 91.44 0)
 			(effects
@@
 			(project "PDU"
 				(path "/e63e39d7-6ac0-4ffd-8aa3-1841a4541b55/12e3318b-d723-448e-80f4-0a2add1fb722"
-					(reference "#PWR0187")
+					(reference "#PWR035")
 					(unit 1)
 				)
@@
 		(on_board yes)
 		(dnp no)
-		(property "Reference" "R12"
+		(property "Reference" "R14"
 			(at 137.414 110.1344 90)
 			(effects
@@
 			(project "PDU"
 				(path "/e63e39d7-6ac0-4ffd-8aa3-1841a4541b55/12e3318b-d723-448e-80f4-0a2add1fb722"
-					(reference "R12")
+					(reference "R14")
 					(unit 1)
 				)
@@
 		(dnp no)
 		(fields_autoplaced yes)
-		(property "Reference" "#PWR0191"
+		(property "Reference" "#PWR033"
 			(at 173.482 81.28 0)
 			(effects
@@
 			(project "PDU"
 				(path "/e63e39d7-6ac0-4ffd-8aa3-1841a4541b55/12e3318b-d723-448e-80f4-0a2add1fb722"
-					(reference "#PWR0191")
+					(reference "#PWR033")
 					(unit 1)
 				)
@@
 		(on_board yes)
 		(dnp no)
-		(property "Reference" "R2"
+		(property "Reference" "R15"
 			(at 228.5787 72.4305 0)
 			(effects
@@
 			(project "PDU"
 				(path "/e63e39d7-6ac0-4ffd-8aa3-1841a4541b55/12e3318b-d723-448e-80f4-0a2add1fb722"
-					(reference "R2")
+					(reference "R15")
 					(unit 1)
 				)
@@
 		(on_board yes)
 		(dnp no)
-		(property "Reference" "#PWR0130"
+		(property "Reference" "#PWR030"
 			(at 138.684 105.156 0)
 			(effects
@@
 			(project "PDU"
 				(path "/e63e39d7-6ac0-4ffd-8aa3-1841a4541b55/12e3318b-d723-448e-80f4-0a2add1fb722"
-					(reference "#PWR0130")
+					(reference "#PWR030")
 					(unit 1)
 				)
@@
 		(on_board yes)
 		(dnp no)
-		(property "Reference" "C50"
+		(property "Reference" "C17"
 			(at 159.512 71.1231 0)
 			(effects
@@
 			(project "PDU"
 				(path "/e63e39d7-6ac0-4ffd-8aa3-1841a4541b55/12e3318b-d723-448e-80f4-0a2add1fb722"
-					(reference "C50")
+					(reference "C17")
 					(unit 1)
 				)
@@
 		(on_board yes)
 		(dnp no)
-		(property "Reference" "R13"
+		(property "Reference" "R16"
 			(at 228.836 81.7997 0)
 			(effects
@@
 			(project "PDU"
 				(path "/e63e39d7-6ac0-4ffd-8aa3-1841a4541b55/12e3318b-d723-448e-80f4-0a2add1fb722"
-					(reference "R13")
+					(reference "R16")
 					(unit 1)
 				)
@@
 		(dnp no)
 		(fields_autoplaced yes)
-		(property "Reference" "#PWR0133"
+		(property "Reference" "#PWR032"
 			(at 153.162 99.06 0)
 			(effects
@@
 			(project "PDU"
 				(path "/e63e39d7-6ac0-4ffd-8aa3-1841a4541b55/12e3318b-d723-448e-80f4-0a2add1fb722"
-					(reference "#PWR0133")
+					(reference "#PWR032")
 					(unit 1)
 				)
@@
 		(dnp no)
 		(fields_autoplaced yes)
-		(property "Reference" "C49"
+		(property "Reference" "C16"
 			(at 121.1961 86.8016 0)
 			(effects
@@
 			(project "PDU"
 				(path "/e63e39d7-6ac0-4ffd-8aa3-1841a4541b55/12e3318b-d723-448e-80f4-0a2add1fb722"
-					(reference "C49")
+					(reference "C16")
 					(unit 1)
 				)
@@
 		(dnp no)
 		(fields_autoplaced yes)
-		(property "Reference" "L5"
+		(property "Reference" "L3"
 			(at 159.512 77.9053 0)
 			(effects
@@
 			(project "PDU"
 				(path "/e63e39d7-6ac0-4ffd-8aa3-1841a4541b55/12e3318b-d723-448e-80f4-0a2add1fb722"
-					(reference "L5")
+					(reference "L3")
 					(unit 1)
 				)
@@
 		(on_board yes)
 		(dnp no)
-		(property "Reference" "#PWR0182"
+		(property "Reference" "#PWR034"
 			(at 205.232 91.44 0)
 			(effects
@@
 			(project "PDU"
 				(path "/e63e39d7-6ac0-4ffd-8aa3-1841a4541b55/12e3318b-d723-448e-80f4-0a2add1fb722"
-					(reference "#PWR0182")
+					(reference "#PWR034")
 					(unit 1)
 				)
@@
 		(dnp no)
 		(fields_autoplaced yes)
-		(property "Reference" "#PWR0188"
+		(property "Reference" "#PWR036"
 			(at 242.062 73.66 0)
 			(effects
@@
 			(project "PDU"
 				(path "/e63e39d7-6ac0-4ffd-8aa3-1841a4541b55/12e3318b-d723-448e-80f4-0a2add1fb722"
-					(reference "#PWR0188")
+					(reference "#PWR036")
 					(unit 1)
 				)
@@
 		(on_board yes)
 		(dnp no)
-		(property "Reference" "C52"
+		(property "Reference" "C19"
 			(at 182.8856 71.8968 0)
 			(effects
@@
 			(project "PDU"
 				(path "/e63e39d7-6ac0-4ffd-8aa3-1841a4541b55/12e3318b-d723-448e-80f4-0a2add1fb722"
-					(reference "C52")
-					(unit 1)
-				)
+					(reference "C19")
+					(unit 1)
+				)

Commit message: cleaned up schematic and bom
Parts:
- C307: renamed from C21; value 0.1uF -> 100nF
- D301: renamed from USBLED1; value WHITE_LED -> LED_WHITE
- R301: renamed from R13; value 14k -> 14kΩ
- R302: renamed from R14; value 5.1k -> 5.1kΩ
- R303: renamed from R15; value 56k -> 56kΩ
- R304: renamed from R16; value 10k -> 10kΩ
- renumbered C15 to C301, C16 to C302, C17 to C303, C18 to C304, C19 to C305, C20 to C306, L3 to L301, U2 to U301, U3 to U302
Other:
- moved on the sheet: D301, R302

Commit message: continued
Parts:
- U302: value SC4215 -> SC4215ASTRT
Changed lines of the file:
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@@
 		(fields_autoplaced yes)
 		(property "Reference" "U302"
-			(at 205.232 63.7372 0)
+			(at 205.232 62.23 0)
 			(effects
 				(font
@@
 			)
 		)
-		(property "Value" "SC4215"
-			(at 205.232 66.2741 0)
+		(property "Value" "SC4215ASTRT"
+			(at 205.232 64.77 0)
 			(effects
 				(font
